Commit message: add wheeled testrig and prismatic joint to lower/raise jetleg

File: jetleg_description/urdf/wheeled_testrig.xacro (robot description, xacro)
@@ -7,6 +7,6 @@
     <xacro:property name="mount_length" value="0.24" />
     <xacro:property name="wheel_length" value="0.04" />
-    <xacro:property name="wheel_radius" value="0.08" />
-    <xacro:property name="wheel_offset" value="0.2" />
+    <xacro:property name="wheel_radius" value="0.15" />
+    <xacro:property name="wheel_offset" value="0.4" />
     <link name="base_link">
     </link>
@@ -60,8 +60,8 @@
                     <cylinder length="${wheel_length}" radius="${wheel_radius}" />
                 </geometry>
-                <contact_coefficients mu="0.5" />
+                <contact_coefficients mu="1.0" />
             </collision>
             <inertial>
-                <mass value="1"/>
+                <mass value="10"/>
                 <inertia ixx="0.001" ixy="0" ixz="0" iyy="0.001" iyz="0" izz="0.001"/>
             </inertial>
@@ -96,8 +96,10 @@
     </link>
     <xacro:include filename="jetleg.xacro"/>
-    <joint name="mount_to_jetleg" type="fixed">
+    <joint name="mount_to_jetleg" type="prismatic">
         <parent link="mount"/>
         <child link="thigh"/>
         <origin xyz="0 0 ${-thigh_length/2}" rpy="0 0 0"/>
+        <axis xyz="0 0 -1" />
+        <limit effort="1000" velocity="10" lower="0" upper="0.3" />
     </joint>
 </robot>

Commit message: change mass of supports in urdf and change control scheme for teleoperation

File: jetleg_description/urdf/wheeled_testrig.xacro (robot description, xacro)
@@ -38,6 +38,6 @@
             </collision>
             <inertial>
-                <mass value="1"/>
-                <inertia ixx="0.001" ixy="0" ixz="0" iyy="0.001" iyz="0" izz="0.001"/>
+                <mass value="50"/>
+                <inertia ixx="0.01" ixy="0" ixz="0" iyy="0.01" iyz="0" izz="0.01"/>
             </inertial>
         </link>
@@ -101,5 +101,5 @@
         <origin xyz="0 0 ${-thigh_length/2}" rpy="0 0 0"/>
         <axis xyz="0 0 -1" />
-        <limit effort="1000" velocity="10" lower="0" upper="0.3" />
+        <limit effort="1000" velocity="10" lower="0" upper="0.6" />
     </joint>
 </robot>

Commit message: add biped model

File: jetleg_description/urdf/wheeled_testrig.xacro (robot description, xacro)
@@ -1,4 +1,4 @@
 <?xml version="1.0"?>
-<robot xmlns:xacro="http://www.ros.org/wiki/xacro" name="jetleg_testrig">
+<robot xmlns:xacro="http://www.ros.org/wiki/xacro" name="jetleg_wheeled_testrig">
     <xacro:include filename="colors.xacro"/>
     <xacro:property name="gantry_height" value="1" />
@@ -10,4 +10,16 @@
     <xacro:property name="wheel_offset" value="0.4" />
     <link name="base_link">
+    </link>
+    <link name="vertical_rail">
+        <visual>
+            <geometry>
+                <box size="0.1 0.1 0.1"/>
+            </geometry>
+            <material name="white"/>
+        </visual>
+        <inertial>
+            <mass value="1"/>
+            <inertia ixx="1" ixy="0" ixz="0" iyy="1" iyz="0" izz="1"/>
+        </inertial>
     </link>
     <link name="gantry">
@@ -38,6 +50,6 @@
             </collision>
             <inertial>
-                <mass value="50"/>
-                <inertia ixx="0.01" ixy="0" ixz="0" iyy="0.01" iyz="0" izz="0.01"/>
+                <mass value="1000"/>
+                <inertia ixx="100" ixy="0" ixz="0" iyy="100" iyz="0" izz="100"/>
             </inertial>
         </link>
@@ -80,8 +92,22 @@
     <xacro:wheel wheelpos="hind_left" parentsupport="left" reflect="1" offset="${-wheel_offset}" />
     <xacro:wheel wheelpos="hind_right" parentsupport="right" reflect="-1" offset="${-wheel_offset}" />
-    <joint name="gantry_to_mount" type="revolute">
+    <joint name="gantry_to_vertical_rail" type="prismatic">
         <origin rpy="0 0 0" xyz="0 0 0"/>
         <parent link="gantry"/>
+        <child link="vertical_rail"/>
+        <limit effort="100" lower="-1" upper="3" velocity="10"/>
+        <axis xyz="0 0 1"/>
+    </joint>
+    <joint name="vertical_rail_to_mount" type="revolute">
+        <origin rpy="0 0 0" xyz="0 -0.1 0"/>
+        <parent link="vertical_rail"/>
         <child link="mount"/>
+        <limit effort="100" lower="${-mount_angle_lim}" upper="${mount_angle_lim}" velocity="10"/>
+        <axis xyz="0 1 0"/>
+    </joint>
+    <joint name="vertical_rail_to_mount_intact" type="revolute">
+        <origin rpy="0 0 0" xyz="0 0.1 0"/>
+        <parent link="vertical_rail"/>
+        <child link="mount_intact"/>
         <limit effort="100" lower="${-mount_angle_lim}" upper="${mount_angle_lim}" velocity="10"/>
         <axis xyz="0 1 0"/>
@@ -95,6 +121,15 @@
         </visual>
     </link>
+    <link name="mount_intact">
+        <visual>
+            <geometry>
+                <cylinder length="${mount_length}" radius="0.08"/>
+            </geometry>
+            <material name="white_transluscent"/>
+        </visual>
+    </link>
     <xacro:include filename="jetleg.xacro"/>
-    <joint name="mount_to_jetleg" type="prismatic">
+    <xacro:include filename="jetleg_intact.xacro"/>
+    <joint name="mount_to_jetleg" type="fixed">
         <parent link="mount"/>
         <child link="thigh"/>
@@ -103,3 +138,10 @@
         <limit effort="1000" velocity="10" lower="0" upper="0.6" />
     </joint>
+    <joint name="mount_to_jetleg_intact" type="fixed">
+        <parent link="mount_intact"/>
+        <child link="thigh_intact"/>
+        <origin xyz="0 0 ${-thigh_intact_length/2}" rpy="0 0 0"/>
+        <axis xyz="0 0 -1" />
+        <limit effort="1000" velocity="10" lower="0" upper="0.6" />
+    </joint>
 </robot>

Commit message: change values in wheeled_testrig

File: jetleg_description/urdf/wheeled_testrig.xacro (robot description, xacro)
@@ -50,5 +50,5 @@
             </collision>
             <inertial>
-                <mass value="50"/>
+                <mass value="500"/>
                 <inertia ixx="10" ixy="0" ixz="0" iyy="10" iyz="0" izz="10"/>
             </inertial>
