Commit message: add stereo camera urdf

File: jetleg_description/urdf/colors.xacro (robot description, xacro)
@@ -1,6 +1,9 @@
 <?xml version="1.0"?>
-<robot xmlns:xacro="http://www.ros.org/wiki/xacro" name="jetleg_testrig">
-   <material name="white">
+<robot xmlns:xacro="http://www.ros.org/wiki/xacro" name="colors">
+    <material name="white">
         <color rgba="1 1 1 1"/>
+    </material>
+    <material name="grey">
+        <color rgba="0.5 0.5 0.5 1"/>
     </material>
     <material name="red">

Commit message: Remove redundant code

File: jetleg_description/urdf/colors.xacro (robot description, xacro)
@@ -3,4 +3,7 @@
     <material name="white">
         <color rgba="1 1 1 1"/>
+    </material>
+    <material name="black">
+        <color rgba="0 0 0 1"/>
     </material>
     <material name="grey">

File: jetleg_description/urdf/stereo_camera.xacro (robot description, xacro)
@@ -10,4 +10,8 @@
                 <material name="black"/>
             </visual>
+            <inertial>
+                <mass value="1" />
+                <inertia ixx="1" ixy="0" ixz="0" iyy="1" iyz="0" izz="1" />
+            </inertial>
         </link>
         <link name="camera_link_right">
@@ -19,4 +23,8 @@
                 <material name="black"/>
             </visual>
+            <inertial>
+                <mass value="1" />
+                <inertia ixx="1" ixy="0" ixz="0" iyy="1" iyz="0" izz="1" />
+            </inertial>
         </link>
         <link name="camera_base">
@@ -28,4 +36,8 @@
                 <material name="grey"/>
             </visual>
+            <inertial>
+                <mass value="1" />
+                <inertia ixx="1" ixy="0" ixz="0" iyy="1" iyz="0" izz="1" />
+            </inertial>
         </link>
         <xacro:insert_block name="joint" />

File: jetleg_description/urdf/testrig_vision.xacro (robot description, xacro)
@@ -1,4 +1,5 @@
 <?xml version="1.0"?>
 <robot xmlns:xacro="http://www.ros.org/wiki/xacro" name="jetleg_testrig_vision">
+    <xacro:include filename="colors.xacro"/>
     <xacro:include filename="$(find jetleg_description)/urdf/wheeled_testrig.xacro"/>
     <xacro:include filename="$(find jetleg_description)/urdf/stereo_camera.xacro"/>

File: jetleg_description/urdf/wheeled_testrig.xacro (robot description, xacro)
@@ -1,5 +1,4 @@
 <?xml version="1.0"?>
 <robot xmlns:xacro="http://www.ros.org/wiki/xacro" name="jetleg_wheeled_testrig">
-    <xacro:include filename="colors.xacro"/>
     <xacro:property name="gantry_height" value="1" />
     <xacro:property name="gantry_width" value="1.6" />
@@ -10,9 +9,4 @@
     <xacro:property name="wheel_offset" value="0.4" />
     <link name="base_link">
-        <inertial>
-                <mass value="1"/>
-                <inertia ixx="1" ixy="0" ixz="0" iyy="1" iyz="0" izz="1"/>
-                <origin rpy="0 0 0" xyz="0 0 0"/>
-        </inertial>
     </link>
     <link name="vertical_rail">
