Commit message: adjust xacro files

File: jetleg_description/urdf/jetleg_single.xacro (robot description, xacro)
@@ -3,29 +3,18 @@
     <xacro:include filename="colors.xacro"/>
     <xacro:include filename="jetleg.xacro"/>
-    <xacro:property name="mount_length" value="0.24" />
     <link name="base_link">
+        <inertial>
+                <mass value="1"/>
+                <inertia ixx="1" ixy="0" ixz="0" iyy="1" iyz="0" izz="1"/>
+                <origin rpy="0 0 0" xyz="0 0 0"/>
+        </inertial>
     </link>
     <!-- Leg Configuration -->
-    <link name="mount">
-        <visual>
-            <geometry>
-                <cylinder length="${mount_length}" radius="0.08"/>
-            </geometry>
-            <material name="white_transluscent"/>
-        </visual>
-    </link>
-    <joint name="base_to_mount" type="fixed">
-        <origin rpy="0 0 0" xyz="0 0 ${mount_length + 1}"/>
+    <joint name="base_to_jetleg" type="fixed">
+        <origin rpy="0 0 0" xyz="0 0 1"/>
         <parent link="base_link"/>
-        <child link="mount"/>
+        <child link="thigh"/>
     </joint>
     <xacro:jetleg identifier="">
     </xacro:jetleg>
-    <joint name="mount_to_jetleg" type="revolute">
-        <parent link="mount"/>
-        <child link="thigh"/>
-        <origin xyz="0 0 ${-thigh_length/2}" rpy="0 0 0"/>
-        <axis xyz="0 1 0" />
-        <limit effort="1000" velocity="10" lower="${-40*pi/180}" upper="${40*pi/180}" />
-    </joint>
 </robot>

File: jetleg_description/urdf/wheeled_testrig.xacro (robot description, xacro)
@@ -10,4 +10,9 @@
     <xacro:property name="wheel_offset" value="0.4" />
     <link name="base_link">
+        <inertial>
+                <mass value="1"/>
+                <inertia ixx="1" ixy="0" ixz="0" iyy="1" iyz="0" izz="1"/>
+                <origin rpy="0 0 0" xyz="0 0 0"/>
+        </inertial>
     </link>
     <link name="vertical_rail">
@@ -30,4 +35,9 @@
             <material name="white_transluscent"/>
         </visual>
+        <inertial>
+                <mass value="1"/>
+                <inertia ixx="1" ixy="0" ixz="0" iyy="1" iyz="0" izz="1"/>
+                <origin rpy="0 0 0" xyz="0 0 0"/>
+        </inertial>
     </link>
     <joint name="base_to_gantry" type="fixed">
@@ -124,4 +134,9 @@
             <material name="white_transluscent"/>
         </visual>
+        <inertial>
+                <mass value="1"/>
+                <inertia ixx="1" ixy="0" ixz="0" iyy="1" iyz="0" izz="1"/>
+                <origin rpy="0 0 0" xyz="0 0 0"/>
+        </inertial>
     </link>
     <link name="mount_intact">
@@ -132,4 +147,9 @@
             <material name="white_transluscent"/>
         </visual>
+        <inertial>
+                <mass value="1"/>
+                <inertia ixx="1" ixy="0" ixz="0" iyy="1" iyz="0" izz="1"/>
+                <origin rpy="0 0 0" xyz="0 0 0"/>
+        </inertial>
     </link>
     <xacro:include filename="jetleg.xacro"/>

Commit message: Restructure xacro files for modularity

File: jetleg_description/urdf/jetleg_single.xacro (robot description, xacro)
@@ -5,7 +5,7 @@
     <link name="base_link">
         <inertial>
-                <mass value="1"/>
-                <inertia ixx="1" ixy="0" ixz="0" iyy="1" iyz="0" izz="1"/>
-                <origin rpy="0 0 0" xyz="0 0 0"/>
+            <mass value="1"/>
+            <inertia ixx="1" ixy="0" ixz="0" iyy="1" iyz="0" izz="1"/>
+            <origin rpy="0 0 0" xyz="0 0 0"/>
         </inertial>
     </link>

File: jetleg_description/urdf/jetleg_testrig_vision.xacro (robot description, xacro)
@@ -1,5 +1,4 @@
 <?xml version="1.0"?>
 <robot xmlns:xacro="http://www.ros.org/wiki/xacro" name="jetleg_testrig_vision">
-    <xacro:include filename="colors.xacro"/>
     <xacro:include filename="$(find jetleg_description)/urdf/wheeled_testrig.xacro"/>
     <xacro:include filename="$(find jetleg_description)/urdf/stereo_camera.xacro"/>

File: jetleg_description/urdf/jetleg_wheeled_testrig.xacro (robot description, xacro)
@@ -1,67 +1,13 @@
 <?xml version="1.0"?>
 <robot xmlns:xacro="http://www.ros.org/wiki/xacro" name="jetleg_wheeled_testrig">
-    <xacro:property name="gantry_height" value="1" />
-    <xacro:property name="gantry_width" value="1.6" />
-    <xacro:property name="mount_angle_lim" value="${40*pi/180}" />
-    <xacro:property name="mount_length" value="0.24" />
+    <!-- Include the basic testrig -->
+    <xacro:include filename="$(find jetleg_description)/urdf/testrig.xacro"/>
+    <!-- Include the JetLeg -->
+    <xacro:include filename="$(find jetleg_description)/urdf/jetleg.xacro"/>
+    <!-- Define reusable variables -->
     <xacro:property name="wheel_length" value="0.04" />
     <xacro:property name="wheel_radius" value="0.15" />
     <xacro:property name="wheel_offset" value="0.4" />
-    <link name="base_link">
-    </link>
-    <link name="vertical_rail">
-        <visual>
-            <geometry>
-                <box size="0.1 0.1 0.1"/>
-            </geometry>
-            <material name="white"/>
-        </visual>
-        <inertial>
-            <mass value="30"/>
-            <inertia ixx="1" ixy="0" ixz="0" iyy="1" iyz="0" izz="1"/>
-        </inertial>
-    </link>
-    <link name="gantry">
-        <visual>
-            <geometry>
-                <box size="0.05 ${gantry_width} 0.05"/>
-            </geometry>
-            <material name="white_transluscent"/>
-        </visual>
-        <inertial>
-            <mass value="1"/>
-            <inertia ixx="1" ixy="0" ixz="0" iyy="1" iyz="0" izz="1"/>
-            <origin rpy="0 0 0" xyz="0 0 0"/>
-        </inertial>
-    </link>
-    <joint name="base_to_gantry" type="fixed">
-        <origin rpy="0 0 0" xyz="0 0 ${gantry_height}"/>
-        <parent link="base_link"/>
-        <child link="gantry"/>
-    </joint>
-    <xacro:macro name="support" params="postfix reflect">
-        <link name="support_${postfix}">
-            <visual>
-                <geometry>
-                    <box size="0.5 0.25 ${gantry_height}"/>
-                </geometry>
-                <material name="red_transluscent"/>
-            </visual>
-            <collision>
-                <geometry>
-                    <box size="0.5 0.25 ${gantry_height}"/>
-                </geometry>
-            </collision>
-            <inertial>
-                <mass value="50"/>
-                <inertia ixx="10" ixy="0" ixz="0" iyy="10" iyz="0" izz="10"/>
-            </inertial>
-        </link>
-        <joint name="gantry_to_support_${postfix}" type="fixed">
-            <parent link="gantry"/>
-            <child link="support_${postfix}"/>
-            <origin xyz="0 ${reflect * gantry_width/2} ${-gantry_height/2}" />
-        </joint>
-    </xacro:macro>
+    <!-- Define the wheel macro -->
     <xacro:macro name="wheel" params="wheelpos parentsupport reflect offset">
         <link name="wheel_${wheelpos}">
@@ -94,31 +40,15 @@
         </joint>
     </xacro:macro>
-    <xacro:support postfix="left" reflect="1" />
-    <xacro:support postfix="right" reflect="-1" />
+    <!-- Create four wheels for the testrig -->
     <xacro:wheel wheelpos="fore_left" parentsupport="left" reflect="1" offset="${wheel_offset}" />
     <xacro:wheel wheelpos="fore_right" parentsupport="right" reflect="-1" offset="${wheel_offset}" />
     <xacro:wheel wheelpos="hind_left" parentsupport="left" reflect="1" offset="${-wheel_offset}" />
     <xacro:wheel wheelpos="hind_right" parentsupport="right" reflect="-1" offset="${-wheel_offset}" />
-    <joint name="gantry_to_vertical_rail" type="prismatic">
-        <origin rpy="0 0 0" xyz="0 0 0"/>
-        <parent link="gantry"/>
-        <child link="vertical_rail"/>
-        <limit effort="100" lower="-1" upper="3" velocity="10"/>
-        <axis xyz="0 0 1"/>
-    </joint>
-    <joint name="vertical_rail_to_mount" type="revolute">
-        <origin rpy="0 0 0" xyz="0 -0.1 0"/>
-        <parent link="vertical_rail"/>
-        <child link="mount"/>
-        <limit effort="100" lower="${-mount_angle_lim}" upper="${mount_angle_lim}" velocity="10"/>
-        <axis xyz="0 1 0"/>
-    </joint>
-    <joint name="vertical_rail_to_mount_intact" type="revolute">
-        <origin rpy="0 0 0" xyz="0 0.1 0"/>
-        <parent link="vertical_rail"/>
-        <child link="mount_intact"/>
-        <limit effort="100" lower="${-mount_angle_lim}" upper="${mount_angle_lim}" velocity="10"/>
-        <axis xyz="0 1 0"/>
-    </joint>
+    <!-- Create two JetLegs -->
+    <xacro:jetleg identifier="">
+    </xacro:jetleg>
+    <xacro:jetleg identifier="_intact">
+    </xacro:jetleg>
+    <!-- Use mounts to attach legs to the testrig -->
     <link name="mount">
         <visual>
@@ -147,9 +77,19 @@
         </inertial>
     </link>
-    <xacro:include filename="jetleg.xacro"/>
-    <xacro:jetleg identifier="">
-    </xacro:jetleg>
-    <xacro:jetleg identifier="_intact">
-    </xacro:jetleg>
+    <!-- Define the additional joints of the robot -->
+    <joint name="vertical_rail_to_mount" type="revolute">
+        <origin rpy="0 0 0" xyz="0 -0.1 0"/>
+        <parent link="vertical_rail"/>
+        <child link="mount"/>
+        <limit effort="100" lower="${-mount_angle_lim}" upper="${mount_angle_lim}" velocity="10"/>
+        <axis xyz="0 1 0"/>
+    </joint>
+    <joint name="vertical_rail_to_mount_intact" type="revolute">
+        <origin rpy="0 0 0" xyz="0 0.1 0"/>
+        <parent link="vertical_rail"/>
+        <child link="mount_intact"/>
+        <limit effort="100" lower="${-mount_angle_lim}" upper="${mount_angle_lim}" velocity="10"/>
+        <axis xyz="0 1 0"/>
+    </joint>
     <joint name="mount_to_jetleg" type="fixed">
         <parent link="mount"/>

File: jetleg_description/urdf/stereo_camera.xacro (robot description, xacro)
@@ -2,4 +2,18 @@
 <robot xmlns:xacro="http://www.ros.org/wiki/xacro" name="stereo_camera">
     <xacro:macro name="stereo_camera" params="baseline *joint">
+        <link name="camera_base">
+            <visual>
+                <geometry>
+                    <box size="0.01 ${baseline+0.02} 0.02"/>
+                </geometry>
+                <origin xyz="0 0 0"/>
+                <material name="grey"/>
+            </visual>
+            <inertial>
+                <mass value="1" />
+                <inertia ixx="1" ixy="0" ixz="0" iyy="1" iyz="0" izz="1" />
+            </inertial>
+        </link>
+        <!-- Links representing the lenses -->
         <link name="camera_link">
             <visual>
@@ -28,17 +42,4 @@
             </inertial>
         </link>
-        <link name="camera_base">
-            <visual>
-                <geometry>
-                    <box size="0.01 ${baseline+0.02} 0.02"/>
-                </geometry>
-                <origin xyz="0 0 0"/>
-                <material name="grey"/>
-            </visual>
-            <inertial>
-                <mass value="1" />
-                <inertia ixx="1" ixy="0" ixz="0" iyy="1" iyz="0" izz="1" />
-            </inertial>
-        </link>
         <xacro:insert_block name="joint" />
         <joint name="camera_base_to_camera_link" type="fixed">

File: jetleg_description/urdf/testrig.xacro (robot description, xacro)
@@ -1,5 +1,5 @@
 <?xml version="1.0"?>
-<robot xmlns:xacro="http://www.ros.org/wiki/xacro" name="jetleg_testrig">
-    <xacro:include filename="colors.xacro"/>
+<robot xmlns:xacro="http://www.ros.org/wiki/xacro" name="testrig">
+    <xacro:include filename="$(find jetleg_description)/urdf/colors.xacro"/>
     <xacro:property name="gantry_height" value="1" />
     <xacro:property name="gantry_width" value="1.6" />
@@ -7,4 +7,16 @@
     <xacro:property name="mount_length" value="0.24" />
     <link name="base_link">
+    </link>
+    <link name="vertical_rail">
+        <visual>
+            <geometry>
+                <box size="0.1 0.1 0.1"/>
+            </geometry>
+            <material name="white"/>
+        </visual>
+        <inertial>
+            <mass value="30"/>
+            <inertia ixx="1" ixy="0" ixz="0" iyy="1" iyz="0" izz="1"/>
+        </inertial>
     </link>
     <link name="gantry">
@@ -16,9 +28,4 @@
         </visual>
     </link>
-    <joint name="base_to_gantry" type="fixed">
-        <origin rpy="0 0 0" xyz="0 0 ${gantry_height}"/>
-        <parent link="base_link"/>
-        <child link="gantry"/>
-    </joint>
     <xacro:macro name="support" params="postfix reflect">
         <link name="support_${postfix}">
@@ -47,28 +54,15 @@
     <xacro:support postfix="left" reflect="1" />
     <xacro:support postfix="right" reflect="-1" />
-    <joint name="gantry_to_mount" type="revolute">
+    <joint name="base_to_gantry" type="fixed">
+        <origin rpy="0 0 0" xyz="0 0 ${gantry_height}"/>
+        <parent link="base_link"/>
+        <child link="gantry"/>
+    </joint>
+    <joint name="gantry_to_vertical_rail" type="prismatic">
         <origin rpy="0 0 0" xyz="0 0 0"/>
         <parent link="gantry"/>
-        <child link="mount"/>
-        <limit effort="100" lower="${-mount_angle_lim}" upper="${mount_angle_lim}" velocity="10"/>
-        <axis xyz="0 1 0"/>
-    </joint>
-    <link name="mount">
-        <visual>
-            <geometry>
-                <cylinder length="${mount_length}" radius="0.08"/>
-            </geometry>
-            <material name="white_transluscent"/>
-        </visual>
-    </link>
-    <xacro:include filename="jetleg.xacro"/>
-    <xacro:jetleg identifier="">
-    </xacro:jetleg>
-    <joint name="mount_to_jetleg" type="fixed">
-        <parent link="mount"/>
-        <child link="thigh"/>
-        <origin xyz="0 0 ${-thigh_length/2}" rpy="0 0 0"/>
-        <axis xyz="0 0 -1" />
-        <limit effort="1000" velocity="10" lower="0" upper="0.6" />
+        <child link="vertical_rail"/>
+        <limit effort="100" lower="-1" upper="3" velocity="10"/>
+        <axis xyz="0 0 1"/>
     </joint>
 </robot>

File: jetleg_description/urdf/testrig_odrive.xacro (robot description, xacro)
@@ -1,5 +1,5 @@
 <?xml version="1.0"?>
 <robot xmlns:xacro="http://www.ros.org/wiki/xacro" name="jetleg_testrig_odrive">
-    <xacro:include filename="$(find jetleg_description)/urdf/testrig.xacro"/>
+    <xacro:include filename="$(find jetleg_description)/urdf/jetleg_testrig.xacro"/>
     <xacro:include filename="$(find jetleg_description)/ros2_control/jetleg.ros2_control.xacro"/>
     <xacro:jetleg_ros2_control name="jetleg_ros2_control"/>
