Commit message: fix camera orientation

File: jetleg_description/urdf/stereo_camera.xacro (robot description, xacro)
@@ -7,5 +7,5 @@
                     <cylinder radius="0.01" length="0.01"/>
                 </geometry>
-                <origin xyz="0 0 0.01"/>
+                <origin xyz="0.01 0 0" rpy="0 ${90*pi/180} 0" />
                 <material name="black"/>
             </visual>
@@ -16,5 +16,5 @@
                     <cylinder radius="0.01" length="0.01"/>
                 </geometry>
-                <origin xyz="0 0 0.01"/>
+                <origin xyz="0.01 0 0" rpy="0 ${90*pi/180} 0" />
                 <material name="black"/>
             </visual>
@@ -33,10 +33,10 @@
             <parent link="camera_base" />
             <child link="camera_link" />
-            <origin xyz="0 ${-baseline/2} 0" rpy="0 ${90*pi/180} 0" />
+            <origin xyz="0 ${-baseline/2} 0"/>
         </joint>
         <joint name="camera_base_to_camera_link_right" type="fixed">
             <parent link="camera_base" />
             <child link="camera_link_right" />
-            <origin xyz="0 ${baseline/2} 0" rpy="0 ${90*pi/180} 0" />
+            <origin xyz="0 ${baseline/2} 0" rpy="0 0 0" />
         </joint>
     </xacro:macro>

File: jetleg_description/urdf/testrig_vision.xacro (robot description, xacro)
@@ -2,5 +2,5 @@
 <robot xmlns:xacro="http://www.ros.org/wiki/xacro" name="jetleg_testrig_odrive">
     <xacro:include filename="$(find jetleg_description)/urdf/testrig.xacro"/>
-    <xacro:include filename="stereo_camera.xacro"/>
+    <xacro:include filename="$(find jetleg_description)/urdf/stereo_camera.xacro"/>
     <xacro:include filename="$(find obstacles)/urdf/prebuilts/staircase_var1.xacro"/>
     <xacro:staircase_var1 postfix="1" offset_x = "2" offset_z = "0.0" />

Commit message: fix issue with frame orientation

File: jetleg_description/urdf/stereo_camera.xacro (robot description, xacro)
@@ -21,5 +21,5 @@
                     <cylinder radius="0.01" length="0.01"/>
                 </geometry>
-                <origin xyz="0.01 0 0" rpy="0 ${90*pi/180} 0" />
+                <origin xyz="0.01 0 0" rpy="0 0 0" />
                 <material name="black"/>
             </visual>
@@ -34,5 +34,5 @@
                     <cylinder radius="0.01" length="0.01"/>
                 </geometry>
-                <origin xyz="0.01 0 0" rpy="0 ${90*pi/180} 0" />
+                <origin xyz="0.01 0 0" rpy="0 0 0" />
                 <material name="black"/>
             </visual>
@@ -46,10 +46,10 @@
             <parent link="camera_base" />
             <child link="camera_link" />
-            <origin xyz="0 ${-baseline/2} 0"/>
+            <origin xyz="0 ${-baseline/2} 0" rpy="${90*pi/180} 0 ${90*pi/180}" />
         </joint>
         <joint name="camera_base_to_camera_link_right" type="fixed">
             <parent link="camera_base" />
             <child link="camera_link_right" />
-            <origin xyz="0 ${baseline/2} 0" rpy="0 0 0" />
+            <origin xyz="0 ${baseline/2} 0" rpy="${90*pi/180} 0 ${90*pi/180}" />
         </joint>
     </xacro:macro>
