Commit message: jetleg rough xacro

File: jetleg_description/urdf/testrig.xacro (robot description, xacro)
@@ -1,19 +1,9 @@
 <?xml version="1.0"?>
 <robot xmlns:xacro="http://www.ros.org/wiki/xacro" name="jetleg_testrig">
-   <material name="white">
-        <color rgba="1 1 1 1"/>
-    </material>
-    <material name="red">
-        <color rgba="1 0 0 1"/>
-    </material>
-    <material name="red_transluscent">
-        <color rgba="1 0 0 0.25"/>
-    </material>
-    <material name="white_transluscent">
-        <color rgba="1 1 1 0.25"/>
-    </material>
+    <xacro:include filename="colors.xacro"/>
     <xacro:property name="gantry_height" value="1" />
     <xacro:property name="gantry_width" value="1.6" />
-    <xacro:property name="mount_angle" value="45*pi/180" />
+    <xacro:property name="mount_angle" value="${25*pi/180}" />
+    <xacro:property name="mount_length" value="0.24" />
     <link name="base_link">
     </link>
@@ -64,6 +54,6 @@
         </joint>
     </xacro:macro>
-    <xacro:support postfix="right" reflect="1" />
-    <xacro:support postfix="left" reflect="-1" />
+    <xacro:support postfix="left" reflect="1" />
+    <xacro:support postfix="right" reflect="-1" />
     <joint name="gantry_to_mount" type="fixed">
         <origin rpy="0 0 0" xyz="0 0.0 0"/>
@@ -74,12 +64,12 @@
         <visual>
             <geometry>
-                <cylinder length="0.24" radius="0.08"/>
+                <cylinder length="${mount_length}" radius="0.08"/>
             </geometry>
-            <material name="white"/>
+            <material name="white_transluscent"/>
             <origin rpy="0 ${mount_angle} 0" xyz="0 0 0"/>
         </visual>
         <collision>
             <geometry>
-                <cylinder length="0.24" radius="0.08"/>
+                <cylinder length="${mount_length}" radius="0.08"/>
             </geometry>
         </collision>
@@ -89,3 +79,9 @@
         </inertial>
     </link>
+    <xacro:include filename="jetleg.xacro"/>
+    <joint name="mount_to_jetleg" type="fixed">
+        <origin rpy="0 ${mount_angle} 0" xyz="${-mount_length*sin(mount_angle)/2} 0 ${-mount_length*cos(mount_angle)/2}"/>
+        <parent link="mount"/>
+        <child link="thigh"/>
+    </joint>
 </robot>

Commit message: add teleoperation for controlling jetleg in pybullet simulation

File: jetleg_description/urdf/testrig.xacro (robot description, xacro)
@@ -21,5 +21,5 @@
         </collision>
         <inertial>
-            <mass value="100"/>
+            <mass value="1000"/>
             <inertia ixx="10" ixy="0" ixz="0" iyy="10" iyz="0" izz="10"/>
         </inertial>
@@ -76,5 +76,5 @@
         </collision>
         <inertial>
-            <mass value="100"/>
+            <mass value="1000"/>
             <inertia ixx="10" ixy="0" ixz="0" iyy="10" iyz="0" izz="10"/>
         </inertial>

Commit message: implement jetleg teleop position control

File: jetleg_description/urdf/testrig.xacro (robot description, xacro)
@@ -15,13 +15,4 @@
             <material name="white_transluscent"/>
         </visual>
-        <collision>
-            <geometry>
-                <box size="0.05 ${gantry_width} 0.05"/>
-            </geometry>
-        </collision>
-        <inertial>
-            <mass value="1000"/>
-            <inertia ixx="10" ixy="0" ixz="0" iyy="10" iyz="0" izz="10"/>
-        </inertial>
     </link>
     <joint name="base_to_gantry" type="fixed">
@@ -44,5 +35,5 @@
             </collision>
             <inertial>
-                <mass value="1000"/>
+                <mass value="10000"/>
                 <inertia ixx="100" ixy="0" ixz="0" iyy="100" iyz="0" izz="100"/>
             </inertial>
@@ -70,13 +61,4 @@
             <material name="white_transluscent"/>
         </visual>
-        <collision>
-            <geometry>
-                <cylinder length="${mount_length}" radius="0.08"/>
-            </geometry>
-        </collision>
-        <inertial>
-            <mass value="1000"/>
-            <inertia ixx="10" ixy="0" ixz="0" iyy="10" iyz="0" izz="10"/>
-        </inertial>
     </link>
     <xacro:include filename="jetleg.xacro"/>

Commit message: changes made to mass and inertia of block

File: jetleg_description/urdf/testrig.xacro (robot description, xacro)
@@ -42,6 +42,6 @@
             </collision>
             <inertial>
-                <mass value="10000"/>
-                <inertia ixx="100" ixy="0" ixz="0" iyy="100" iyz="0" izz="100"/>
+                <mass value="1000"/>
+                <inertia ixx="1" ixy="0" ixz="0" iyy="1" iyz="0" izz="1"/>
             </inertial>
         </link>

Commit message: add moveit config package for jetleg

File: jetleg_description/urdf/testrig.xacro (robot description, xacro)
@@ -42,6 +42,6 @@
             </collision>
             <inertial>
-                <mass value="1000"/>
-                <inertia ixx="1" ixy="0" ixz="0" iyy="1" iyz="0" izz="1"/>
+                <mass value="100"/>
+                <inertia ixx="10" ixy="0" ixz="0" iyy="10" iyz="0" izz="10"/>
             </inertial>
         </link>

Commit message: add inertial info to testrig model

File: jetleg_description/urdf/testrig.xacro (robot description, xacro)
@@ -27,4 +27,8 @@
             <material name="white_transluscent"/>
         </visual>
+        <inertial>
+            <mass value="1"/>
+            <inertia ixx="1" ixy="0" ixz="0" iyy="1" iyz="0" izz="1"/>
+        </inertial>
     </link>
     <xacro:macro name="support" params="postfix reflect">

Commit message: [Config] Test impedance controller with Gazebo

File: jetleg_description/urdf/testrig.xacro (robot description, xacro)
@@ -72,10 +72,10 @@
         <child link="gantry"/>
     </joint>
-    <joint name="gantry_to_vertical_rail" type="prismatic">
+    <joint name="gantry_to_vertical_rail" type="fixed">
         <origin rpy="0 0 0" xyz="0 0 0"/>
         <parent link="gantry"/>
         <child link="vertical_rail"/>
-        <limit effort="100" lower="-0.5" upper="0.0" velocity="10"/>
-        <axis xyz="0 0 1"/>
+        <!-- <limit effort="100" lower="-0.5" upper="0.0" velocity="10"/>
+        <axis xyz="0 0 1"/> -->
     </joint>
 </robot>

File: jetleg_moveit_config/config/jetleg_wheeled_testrig.ros2_control.xacro (robot description, xacro)
@@ -6,9 +6,9 @@
             <hardware>
                 <!-- By default, set up controllers for simulation. This won't work on real hardware -->
-                <!-- <plugin>gazebo_ros2_control/GazeboSystem</plugin> -->
-                <plugin>fake_effort_interface/GenericSystem</plugin>
+                <plugin>gazebo_ros2_control/GazeboSystem</plugin>
+                <!-- <plugin>fake_effort_interface/GenericSystem</plugin> -->
             </hardware>
             <joint name="vertical_rail_to_mount">
-                <command_interface name="acceleration"/>
+                <command_interface name="effort"/>
                 <state_interface name="position">
                   <param name="initial_value">${initial_positions['vertical_rail_to_mount']}</param>
@@ -17,5 +17,5 @@
             </joint>
             <joint name="knee_joint">
-                <command_interface name="acceleration"/>
+                <command_interface name="effort"/>
                 <state_interface name="position">
                   <param name="initial_value">${initial_positions['knee_joint']}</param>
@@ -24,5 +24,5 @@
             </joint>
             <joint name="ankle_joint">
-                <command_interface name="acceleration"/>
+                <command_interface name="effort"/>
                 <state_interface name="position">
                   <param name="initial_value">${initial_positions['ankle_joint']}</param>
@@ -31,5 +31,5 @@
             </joint>
             <joint name="vertical_rail_to_mount_intact">
-                <command_interface name="acceleration"/>
+                <command_interface name="effort"/>
                 <state_interface name="position">
                   <param name="initial_value">${initial_positions['vertical_rail_to_mount_intact']}</param>
@@ -38,5 +38,5 @@
             </joint>
             <joint name="knee_joint_intact">
-                <command_interface name="acceleration"/>
+                <command_interface name="effort"/>
                 <state_interface name="position">
                   <param name="initial_value">${initial_positions['knee_joint_intact']}</param>
@@ -45,5 +45,5 @@
             </joint>
             <joint name="ankle_joint_intact">
-                <command_interface name="acceleration"/>
+                <command_interface name="effort"/>
                 <state_interface name="position">
                   <param name="initial_value">${initial_positions['ankle_joint_intact']}</param>
@@ -84,5 +84,5 @@
                 </state_interface>
             </joint>
-            <joint name="gantry_to_vertical_rail">
+            <!-- <joint name="gantry_to_vertical_rail">
                 <state_interface name="position">
                   <param name="initial_value">0.0</param>
@@ -91,5 +91,5 @@
                   <param name="initial_value">0.0</param>
                 </state_interface>
-            </joint>
+            </joint> -->
         </ros2_control>
     </xacro:macro>

File: jetleg_moveit_config/config/jetleg_wheeled_testrig.urdf.xacro (robot description, xacro)
@@ -6,4 +6,4 @@
     <!-- Import control_xacro -->
     <xacro:include filename="jetleg_wheeled_testrig.ros2_control.xacro" />
-    <xacro:jetleg_wheeled_testrig_ros2_control name="GazeboSystem" initial_positions_file="$(arg initial_positions_file)"/>
+    <xacro:jetleg_wheeled_testrig_ros2_control name="JetlegSystem" initial_positions_file="$(arg initial_positions_file)"/>
 </robot>
