Commit message: testrig mount is now a revolute joint

File: jetleg_description/urdf/jetleg.xacro (robot description, xacro)
@@ -50,5 +50,5 @@
         <child link="shank"/>
         <axis xyz="0 1 0"/>
-        <limit effort="100" lower="-1.5" upper="0.0" velocity="10"/>
+        <limit effort="100" lower="0.0" upper="1.5" velocity="10"/>
     </joint>
     <link name="foot">
@@ -58,5 +58,5 @@
             </geometry>
             <material name="white"/>
-            <origin xyz="${-(foot_length/2-0.05)} 0 ${-ankle_joint_radius-foot_height/2}"/>
+            <origin xyz="${(foot_length/2-0.05)} 0 ${-ankle_joint_radius-foot_height/2}"/>
         </visual>
         <collision>
@@ -64,10 +64,10 @@
                 <box size="${foot_length} ${foot_width} ${foot_height}"/>
             </geometry>
-            <origin xyz="${-(foot_length/2-0.05)} 0 ${-ankle_joint_radius-foot_height/2}"/>
+            <origin xyz="${(foot_length/2-0.05)} 0 ${-ankle_joint_radius-foot_height/2}"/>
         </collision>
         <inertial>
             <mass value="10"/>
             <inertia ixx="1" ixy="0" ixz="0" iyy="1" iyz="0" izz="1"/>
-            <origin xyz="${-(foot_length/2-0.05)} 0 ${-ankle_joint_radius-foot_height/2}"/>
+            <origin xyz="${(foot_length/2-0.05)} 0 ${-ankle_joint_radius-foot_height/2}"/>
         </inertial>
     </link>
@@ -77,5 +77,5 @@
         <child link="foot"/>
         <axis xyz="0 1 0"/>
-        <limit effort="100" lower="-0.5" upper="0.1" velocity="10"/>
+        <limit effort="100" lower="-0.1" upper="0.5" velocity="10"/>
     </joint>
 </robot>

File: jetleg_description/urdf/testrig.urdf (robot description, URDF)
Before this commit: robot jetleg_testrig, 4 links, 3 joints
Links:
- removed link base_two
- added link foot, mass 10; collision box size=0.3 0.1 0.05; visual box size=0.3 0.1 0.05
- added link shank, mass 10; collision cylinder length=0.3 radius=0.06; visual cylinder length=0.3 radius=0.06
- added link support_left, mass 1000; collision box size=0.5 0.25 1; visual box size=0.5 0.25 1
- added link support_right, mass 1000; collision box size=0.5 0.25 1; visual box size=0.5 0.25 1
- added link thigh, mass 10; collision cylinder length=0.3 radius=0.06; visual cylinder length=0.3 radius=0.06
- link base_link: mass 1000 -> None; geometry 
- link gantry: geometry collision box size=0.05 1.6 0.05; visual box size=0.05 1.6 0.05
Joints:
- removed joint gantry_to_base2
- added joint ankle_joint: type revolute, parent shank, child foot, origin xyz=0 0 -0.35000000000000003 rpy=0 0 0, axis 0 1 0, limit lower=-0.5 upper=0.1 effort=100 velocity=10
- added joint gantry_to_support_left: type fixed, parent gantry, child support_left, origin xyz=0 0.8 -0.5
- added joint gantry_to_support_right: type fixed, parent gantry, child support_right, origin xyz=0 -0.8 -0.5
- added joint knee_joint: type revolute, parent thigh, child shank, origin xyz=0 0 -0.175 rpy=0 0 0, axis 0 1 0, limit lower=-1.5 upper=0.0 effort=100 velocity=10
- added joint mount_to_jetleg: type fixed, parent mount, child thigh, origin xyz=0 0 -0.15 rpy=0 0 0
- joint base_to_gantry: origin xyz=0 -0.8 0.4 rpy=0 0 0 -> xyz=0 0 1 rpy=0 0 0
- joint gantry_to_mount: limit (none) -> lower=-0.6981317007977318 upper=0.6981317007977318 effort=100; type fixed -> revolute

File: jetleg_description/urdf/testrig.xacro (robot description, xacro)
@@ -4,5 +4,5 @@
     <xacro:property name="gantry_height" value="1" />
     <xacro:property name="gantry_width" value="1.6" />
-    <xacro:property name="mount_angle" value="${25*pi/180}" />
+    <xacro:property name="mount_angle_lim" value="${40*pi/180}" />
     <xacro:property name="mount_length" value="0.24" />
     <link name="base_link">
@@ -51,13 +51,15 @@
             <parent link="gantry"/>
             <child link="support_${postfix}"/>
-            <origin xyz="0 ${reflect * gantry_width/2} -${gantry_height/2}" />
+            <origin xyz="0 ${reflect * gantry_width/2} ${-gantry_height/2}" />
         </joint>
     </xacro:macro>
     <xacro:support postfix="left" reflect="1" />
     <xacro:support postfix="right" reflect="-1" />
-    <joint name="gantry_to_mount" type="fixed">
-        <origin rpy="0 0 0" xyz="0 0.0 0"/>
+    <joint name="gantry_to_mount" type="revolute">
+        <origin rpy="0 0 0" xyz="0 0 0"/>
         <parent link="gantry"/>
         <child link="mount"/>
+        <limit effort="100" lower="${-mount_angle_lim}" upper="${mount_angle_lim}" velocity="10"/>
+        <axis xyz="0 1 0"/>
     </joint>
     <link name="mount">
@@ -67,5 +69,4 @@
             </geometry>
             <material name="white_transluscent"/>
-            <origin rpy="0 ${mount_angle} 0" xyz="0 0 0"/>
         </visual>
         <collision>
@@ -81,7 +82,7 @@
     <xacro:include filename="jetleg.xacro"/>
     <joint name="mount_to_jetleg" type="fixed">
-        <origin rpy="0 ${mount_angle} 0" xyz="${-mount_length*sin(mount_angle)/2} 0 ${-mount_length*cos(mount_angle)/2}"/>
         <parent link="mount"/>
         <child link="thigh"/>
+        <origin xyz="0 0 ${-thigh_length/2}" rpy="0 0 0"/>
     </joint>
 </robot>

Commit message: generate gait on both legs

File: jetleg_description/urdf/jetleg.xacro (robot description, xacro)
@@ -1,6 +1,6 @@
 <?xml version="1.0"?>
 <robot xmlns:xacro="http://www.ros.org/wiki/xacro" name="jetleg">
-    <xacro:property name="thigh_length" value="0.3" />
-    <xacro:property name="shank_length" value="0.3" />
+    <xacro:property name="thigh_length" value="0.5" />
+    <xacro:property name="shank_length" value="0.4" />
     <xacro:property name="knee_joint_radius" value="0.025" />
     <xacro:property name="ankle_joint_radius" value="0.025" />
@@ -21,5 +21,5 @@
         </collision>
         <inertial>
-            <mass value="10"/>
+            <mass value="20"/>
             <inertia ixx="1" ixy="0" ixz="0" iyy="1" iyz="0" izz="1"/>
         </inertial>
@@ -67,5 +67,5 @@
         </collision>
         <inertial>
-            <mass value="10"/>
+            <mass value="1.5"/>
             <inertia ixx="1" ixy="0" ixz="0" iyy="1" iyz="0" izz="1"/>
             <origin xyz="${(foot_length/2-0.05)} 0 ${-ankle_joint_radius-foot_height/2}"/>

File: jetleg_description/urdf/jetleg_intact.xacro (robot description, xacro)
@@ -1,6 +1,6 @@
 <?xml version="1.0"?>
 <robot xmlns:xacro="http://www.ros.org/wiki/xacro" name="jetleg_intact">
-    <xacro:property name="thigh_intact_length" value="0.3" />
-    <xacro:property name="shank_intact_length" value="0.3" />
+    <xacro:property name="thigh_intact_length" value="0.5" />
+    <xacro:property name="shank_intact_length" value="0.4" />
     <xacro:property name="knee_intact_joint_radius" value="0.025" />
     <xacro:property name="ankle_intact_joint_radius" value="0.025" />
@@ -21,5 +21,5 @@
         </collision>
         <inertial>
-            <mass value="10"/>
+            <mass value="20"/>
             <inertia ixx="1" ixy="0" ixz="0" iyy="1" iyz="0" izz="1"/>
         </inertial>
@@ -67,5 +67,5 @@
         </collision>
         <inertial>
-            <mass value="10"/>
+            <mass value="1.5"/>
             <inertia ixx="1" ixy="0" ixz="0" iyy="1" iyz="0" izz="1"/>
             <origin xyz="${(foot_intact_length/2-0.05)} 0 ${-ankle_intact_joint_radius-foot_intact_height/2}"/>

File: jetleg_description/urdf/wheeled_testrig.xacro (robot description, xacro)
@@ -19,5 +19,5 @@
         </visual>
         <inertial>
-            <mass value="1"/>
+            <mass value="30"/>
             <inertia ixx="1" ixy="0" ixz="0" iyy="1" iyz="0" izz="1"/>
         </inertial>
@@ -50,6 +50,6 @@
             </collision>
             <inertial>
-                <mass value="1000"/>
-                <inertia ixx="100" ixy="0" ixz="0" iyy="100" iyz="0" izz="100"/>
+                <mass value="50"/>
+                <inertia ixx="10" ixy="0" ixz="0" iyy="10" iyz="0" izz="10"/>
             </inertial>
         </link>

Commit message: Merge branch 'gait_generation' into ab_devel

File: jetleg_description/urdf/jetleg.xacro (robot description, xacro)
@@ -8,77 +8,79 @@
     <xacro:property name="foot_width" value="0.1" />
     <xacro:property name="foot_height" value="0.05" />
-    <link name="thigh">
-        <visual>
-            <geometry>
-                <cylinder length="${thigh_length}" radius="0.06"/>
-            </geometry>
-            <material name="white"/>
-        </visual>
-        <collision>
-            <geometry>
-                <cylinder length="${thigh_length}" radius="0.06"/>
-            </geometry>
-        </collision>
-        <inertial>
-            <mass value="20"/>
-            <inertia ixx="1" ixy="0" ixz="0" iyy="1" iyz="0" izz="1"/>
-        </inertial>
-    </link>
-    <link name="shank">
-        <visual>
-            <geometry>
-                <cylinder length="${shank_length}" radius="0.06"/>
-            </geometry>
-            <material name="white"/>
-            <origin rpy="0 0 0" xyz="0 0 ${-shank_length/2-knee_joint_radius}"/>
-        </visual>
-        <collision>
-            <geometry>
-                <cylinder length="${shank_length}" radius="0.06"/>
-            </geometry>
-            <origin rpy="0 0 0" xyz="0 0 ${-shank_length/2-knee_joint_radius}"/>
-        </collision>
-        <inertial>
-            <mass value="10"/>
-            <inertia ixx="1" ixy="0" ixz="0" iyy="1" iyz="0" izz="1"/>
-            <origin rpy="0 0 0" xyz="0 0 ${-shank_length/2-knee_joint_radius}"/>
-        </inertial>
-    </link>
-    <joint name="knee_joint" type="revolute">
-        <origin rpy="0 0 0" xyz="0 0 ${-thigh_length/2-knee_joint_radius}"/>
-        <parent link="thigh"/>
-        <child link="shank"/>
-        <axis xyz="0 1 0"/>
-        <limit effort="100" lower="0.0" upper="1.5" velocity="10"/>
-    </joint>
-    <link name="foot">
-        <contact>
-            <lateral_friction value="100"/>
-        </contact>
-        <visual>
-            <geometry>
-                <box size="${foot_length} ${foot_width} ${foot_height}"/>
-            </geometry>
-            <material name="white"/>
-            <origin xyz="${(foot_length/2-0.05)} 0 ${-ankle_joint_radius-foot_height/2}"/>
-        </visual>
-        <collision>
-            <geometry>
-                <box size="${foot_length} ${foot_width} ${foot_height}"/>
-            </geometry>
-            <origin xyz="${(foot_length/2-0.05)} 0 ${-ankle_joint_radius-foot_height/2}"/>
-        </collision>
-        <inertial>
-            <mass value="1.5"/>
-            <inertia ixx="1" ixy="0" ixz="0" iyy="1" iyz="0" izz="1"/>
-            <origin xyz="${(foot_length/2-0.05)} 0 ${-ankle_joint_radius-foot_height/2}"/>
-        </inertial>
-    </link>
-    <joint name="ankle_joint" type="revolute">
-        <origin rpy="0 0 0" xyz="0 0 ${-(knee_joint_radius + shank_length + ankle_joint_radius)}"/>
-        <parent link="shank"/>
-        <child link="foot"/>
-        <axis xyz="0 1 0"/>
-        <limit effort="100" lower="-0.1" upper="0.5" velocity="10"/>
-    </joint>
+    <xacro:macro name="jetleg" params="identifier">
+        <link name="thigh${identifier}">
+            <visual>
+                <geometry>
+                    <cylinder length="${thigh_length}" radius="0.06"/>
+                </geometry>
+                <material name="white"/>
+            </visual>
+            <collision>
+                <geometry>
+                    <cylinder length="${thigh_length}" radius="0.06"/>
+                </geometry>
+            </collision>
+            <inertial>
+                <mass value="20"/>
+                <inertia ixx="1" ixy="0" ixz="0" iyy="1" iyz="0" izz="1"/>
+            </inertial>
+        </link>
+        <link name="shank${identifier}">
+            <visual>
+                <geometry>
+                    <cylinder length="${shank_length}" radius="0.06"/>
+                </geometry>
+                <material name="white"/>
+                <origin rpy="0 0 0" xyz="0 0 ${-shank_length/2-knee_joint_radius}"/>
+            </visual>
+            <collision>
+                <geometry>
+                    <cylinder length="${shank_length}" radius="0.06"/>
+                </geometry>
+                <origin rpy="0 0 0" xyz="0 0 ${-shank_length/2-knee_joint_radius}"/>
+            </collision>
+            <inertial>
+                <mass value="10"/>
+                <inertia ixx="1" ixy="0" ixz="0" iyy="1" iyz="0" izz="1"/>
+                <origin rpy="0 0 0" xyz="0 0 ${-shank_length/2-knee_joint_radius}"/>
+            </inertial>
+        </link>
+        <joint name="knee_joint${identifier}" type="revolute">
+            <origin rpy="0 0 0" xyz="0 0 ${-thigh_length/2-knee_joint_radius}"/>
+            <parent link="thigh${identifier}"/>
+            <child link="shank${identifier}"/>
+            <axis xyz="0 1 0"/>
+            <limit effort="100" lower="0.0" upper="1.5" velocity="10"/>
+        </joint>
+        <link name="foot${identifier}">
+            <contact>
+                <lateral_friction value="100"/>
+            </contact>
+            <visual>
+                <geometry>
+                    <box size="${foot_length} ${foot_width} ${foot_height}"/>
+                </geometry>
+                <material name="white"/>
+                <origin xyz="${(foot_length/2-0.05)} 0 ${-ankle_joint_radius-foot_height/2}"/>
+            </visual>
+            <collision>
+                <geometry>
+                    <box size="${foot_length} ${foot_width} ${foot_height}"/>
+                </geometry>
+                <origin xyz="${(foot_length/2-0.05)} 0 ${-ankle_joint_radius-foot_height/2}"/>
+            </collision>
+            <inertial>
+                <mass value="1.5"/>
+                <inertia ixx="1" ixy="0" ixz="0" iyy="1" iyz="0" izz="1"/>
+                <origin xyz="${(foot_length/2-0.05)} 0 ${-ankle_joint_radius-foot_height/2}"/>
+            </inertial>
+        </link>
+        <joint name="ankle_joint${identifier}" type="revolute">
+            <origin rpy="0 0 0" xyz="0 0 ${-(knee_joint_radius + shank_length + ankle_joint_radius)}"/>
+            <parent link="shank${identifier}"/>
+            <child link="foot${identifier}"/>
+            <axis xyz="0 1 0"/>
+            <limit effort="100" lower="-0.1" upper="0.5" velocity="10"/>
+        </joint>
+    </xacro:macro>
 </robot>

File: jetleg_description/urdf/testrig.xacro (robot description, xacro)
@@ -63,4 +63,6 @@
     </link>
     <xacro:include filename="jetleg.xacro"/>
+    <xacro:jetleg identifer="">
+    </xacro:jetleg>
     <joint name="mount_to_jetleg" type="fixed">
         <parent link="mount"/>

File: jetleg_description/urdf/wheeled_testrig.xacro (robot description, xacro)
@@ -134,5 +134,8 @@
     </link>
     <xacro:include filename="jetleg.xacro"/>
-    <xacro:include filename="jetleg_intact.xacro"/>
+    <xacro:jetleg identifier="">
+    </xacro:jetleg>
+    <xacro:jetleg identifier="_intact">
+    </xacro:jetleg>
     <joint name="mount_to_jetleg" type="fixed">
         <parent link="mount"/>
@@ -145,5 +148,5 @@
         <parent link="mount_intact"/>
         <child link="thigh_intact"/>
-        <origin xyz="0 0 ${-thigh_intact_length/2}" rpy="0 0 0"/>
+        <origin xyz="0 0 ${-thigh_length/2}" rpy="0 0 0"/>
         <axis xyz="0 0 -1" />
         <limit effort="1000" velocity="10" lower="0" upper="0.6" />

Commit message: add bipedal xacro, generalize launch and config files for reuse

File: jetleg_description/urdf/jetleg.xacro (robot description, xacro)
@@ -8,4 +8,7 @@
     <xacro:property name="foot_width" value="0.1" />
     <xacro:property name="foot_height" value="0.05" />
+    <xacro:property name="thigh_mass" value="20" />
+    <xacro:property name="shank_mass" value="10" />
+    <xacro:property name="foot_mass" value="1.5" />
     <xacro:macro name="jetleg" params="identifier">
         <link name="thigh${identifier}">
@@ -22,6 +25,6 @@
             </collision>
             <inertial>
-                <mass value="20"/>
-                <inertia ixx="1" ixy="0" ixz="0" iyy="1" iyz="0" izz="1"/>
+                <mass value="${thigh_mass}"/>
+                <inertia ixx="${thigh_mass/12*(3*0.06**2+thigh_length**2)}" ixy="0" ixz="0" iyy="${thigh_mass/12*(3*0.06**2+thigh_length**2)}" iyz="0" izz="${0.5*thigh_mass*0.06**2}"/>
             </inertial>
         </link>
@@ -41,6 +44,6 @@
             </collision>
             <inertial>
-                <mass value="10"/>
-                <inertia ixx="1" ixy="0" ixz="0" iyy="1" iyz="0" izz="1"/>
+                <mass value="${shank_mass}"/>
+                <inertia ixx="${shank_mass/12*(3*0.06**2+shank_length**2)}" ixy="0" ixz="0" iyy="${shank_mass/12*(3*0.06**2+shank_length**2)}" iyz="0" izz="${0.5*shank_mass*0.06**2}"/>
                 <origin rpy="0 0 0" xyz="0 0 ${-shank_length/2-knee_joint_radius}"/>
             </inertial>

File: jetleg_description/urdf/testrig.xacro (robot description, xacro)
@@ -63,5 +63,5 @@
     </link>
     <xacro:include filename="jetleg.xacro"/>
-    <xacro:jetleg identifer="">
+    <xacro:jetleg identifier="">
     </xacro:jetleg>
     <joint name="mount_to_jetleg" type="fixed">
@@ -69,4 +69,6 @@
         <child link="thigh"/>
         <origin xyz="0 0 ${-thigh_length/2}" rpy="0 0 0"/>
+        <axis xyz="0 0 -1" />
+        <limit effort="1000" velocity="10" lower="0" upper="0.6" />
     </joint>
 </robot>

Commit message: Prepare environment single leg control

File: jetleg_description/urdf/jetleg.xacro (robot description, xacro)
@@ -54,5 +54,5 @@
             <child link="shank${identifier}"/>
             <axis xyz="0 1 0"/>
-            <limit effort="100" lower="0.0" upper="1.5" velocity="10"/>
+            <limit effort="100" lower="0.0" upper="2.5" velocity="10"/>
         </joint>
         <link name="foot${identifier}">

Commit message: Add functionality for running saved RL models

File: jetleg_description/urdf/jetleg.xacro (robot description, xacro)
@@ -25,7 +25,7 @@
             </collision>
             <inertial>
-                <mass value="${thigh_mass}"/>
-                <inertia ixx="${thigh_mass/12*(3*0.06**2+thigh_length**2)}" ixy="0" ixz="0" iyy="${thigh_mass/12*(3*0.06**2+thigh_length**2)}" iyz="0" izz="${0.5*thigh_mass*0.06**2}"/>
-            </inertial>
+            <mass value="${thigh_mass}"/>
+            <inertia ixx="1" ixy="0" ixz="0" iyy="1" iyz="0" izz="1"/>
+        </inertial>
         </link>
         <link name="shank${identifier}">
@@ -45,5 +45,5 @@
             <inertial>
                 <mass value="${shank_mass}"/>
-                <inertia ixx="${shank_mass/12*(3*0.06**2+shank_length**2)}" ixy="0" ixz="0" iyy="${shank_mass/12*(3*0.06**2+shank_length**2)}" iyz="0" izz="${0.5*shank_mass*0.06**2}"/>
+                <inertia ixx="1" ixy="0" ixz="0" iyy="1" iyz="0" izz="1"/>
                 <origin rpy="0 0 0" xyz="0 0 ${-shank_length/2-knee_joint_radius}"/>
             </inertial>
@@ -74,5 +74,5 @@
             </collision>
             <inertial>
-                <mass value="1.5"/>
+                <mass value="${foot_mass}"/>
                 <inertia ixx="1" ixy="0" ixz="0" iyy="1" iyz="0" izz="1"/>
                 <origin xyz="${(foot_length/2-0.05)} 0 ${-ankle_joint_radius-foot_height/2}"/>

File: jetleg_description/urdf/wheeled_testrig.xacro (robot description, xacro)
@@ -36,7 +36,7 @@
         </visual>
         <inertial>
-                <mass value="1"/>
-                <inertia ixx="1" ixy="0" ixz="0" iyy="1" iyz="0" izz="1"/>
-                <origin rpy="0 0 0" xyz="0 0 0"/>
+            <mass value="1"/>
+            <inertia ixx="1" ixy="0" ixz="0" iyy="1" iyz="0" izz="1"/>
+            <origin rpy="0 0 0" xyz="0 0 0"/>
         </inertial>
     </link>
@@ -60,5 +60,5 @@
             </collision>
             <inertial>
-                <mass value="500"/>
+                <mass value="50"/>
                 <inertia ixx="10" ixy="0" ixz="0" iyy="10" iyz="0" izz="10"/>
             </inertial>

Commit message: fix moveit configurations for wheeled_testrig

File: jetleg_description/urdf/jetleg.xacro (robot description, xacro)
@@ -54,5 +54,5 @@
             <child link="shank${identifier}"/>
             <axis xyz="0 1 0"/>
-            <limit effort="100" lower="0.0" upper="2.5" velocity="10"/>
+            <limit effort="100" lower="0.0" upper="2.5" velocity="10.0"/>
         </joint>
         <link name="foot${identifier}">
@@ -84,5 +84,5 @@
             <child link="foot${identifier}"/>
             <axis xyz="0 1 0"/>
-            <limit effort="100" lower="-0.1" upper="0.5" velocity="10"/>
+            <limit effort="100" lower="-0.1" upper="0.5" velocity="10.0"/>
         </joint>
     </xacro:macro>
