Commit message: add material description to models

File: jetleg_description/urdf/jetleg.xacro (robot description, xacro)
@@ -29,4 +29,7 @@
         </inertial>
         </link>
+        <gazebo reference="thigh${identifier}">
+            <material>Gazebo/White</material>
+        </gazebo>
         <link name="shank${identifier}">
             <visual>
@@ -49,4 +52,7 @@
             </inertial>
         </link>
+        <gazebo reference="shank${identifier}">
+            <material>Gazebo/White</material>
+        </gazebo>
         <joint name="knee_joint${identifier}" type="revolute">
             <origin rpy="0 0 0" xyz="0 0 ${-thigh_length/2-knee_joint_radius}"/>
@@ -79,4 +85,7 @@
             </inertial>
         </link>
+        <gazebo reference="foot${identifier}">
+            <material>Gazebo/White</material>
+        </gazebo>
         <joint name="ankle_joint${identifier}" type="revolute">
             <origin rpy="0 0 0" xyz="0 0 ${-(knee_joint_radius + shank_length + ankle_joint_radius)}"/>

File: jetleg_description/urdf/jetleg_testrig.xacro (robot description, xacro)
@@ -10,7 +10,10 @@
                 <cylinder length="${mount_length}" radius="0.08"/>
             </geometry>
-            <material name="white_transluscent"/>
+            <material name="black"/>
         </visual>
     </link>
+    <gazebo reference="mount">
+        <material>Gazebo/Black</material>
+    </gazebo>
     <joint name="vertical_rail_to_mount" type="revolute">
         <origin rpy="0 0 0" xyz="0 0 0"/>

File: jetleg_description/urdf/jetleg_wheeled_testrig.xacro (robot description, xacro)
@@ -56,5 +56,5 @@
                 <cylinder length="${mount_length}" radius="0.08"/>
             </geometry>
-            <material name="white_transluscent"/>
+            <material name="black"/>
         </visual>
         <inertial>
@@ -64,4 +64,7 @@
         </inertial>
     </link>
+    <gazebo reference="mount">
+        <material>Gazebo/Black</material>
+    </gazebo>
     <link name="mount_intact">
         <visual>
@@ -69,5 +72,5 @@
                 <cylinder length="${mount_length}" radius="0.08"/>
             </geometry>
-            <material name="white_transluscent"/>
+            <material name="black"/>
         </visual>
         <inertial>
@@ -77,4 +80,7 @@
         </inertial>
     </link>
+    <gazebo reference="mount_intact">
+        <material>Gazebo/Black</material>
+    </gazebo>
     <!-- Define the additional joints of the robot -->
     <joint name="vertical_rail_to_mount" type="revolute">

File: jetleg_description/urdf/stereo_camera.xacro (robot description, xacro)
@@ -16,4 +16,7 @@
             </inertial>
         </link>
+        <gazebo reference="camera_base">
+            <material>Gazebo/Grey</material>
+        </gazebo>
         <!-- Links representing the lenses -->
         <link name="camera_link">
@@ -43,4 +46,10 @@
             </inertial>
         </link>
+        <gazebo reference="camera_link">
+            <material>Gazebo/Black</material>
+        </gazebo>
+        <gazebo reference="camera_link_right">
+            <material>Gazebo/Black</material>
+        </gazebo>
         <xacro:insert_block name="joint" />
         <joint name="camera_base_to_camera_link" type="fixed">

File: jetleg_description/urdf/testrig.xacro (robot description, xacro)
@@ -20,4 +20,7 @@
         </inertial>
     </link>
+    <gazebo reference="vertical_rail">
+        <material>Gazebo/White</material>
+    </gazebo>
     <link name="gantry">
         <visual>
@@ -25,5 +28,5 @@
                 <box size="0.05 ${gantry_width} 0.05"/>
             </geometry>
-            <material name="white_transluscent"/>
+            <material name="white"/>
         </visual>
         <inertial>
@@ -32,4 +35,7 @@
         </inertial>
     </link>
+    <gazebo reference="gantry">
+        <material>Gazebo/White</material>
+    </gazebo>
     <xacro:macro name="support" params="postfix reflect">
         <link name="support_${postfix}">
@@ -38,5 +44,5 @@
                     <box size="0.5 0.25 ${gantry_height}"/>
                 </geometry>
-                <material name="red_transluscent"/>
+                <material name="red"/>
             </visual>
             <collision>
@@ -50,4 +56,7 @@
             </inertial>
         </link>
+        <gazebo reference="support_${postfix}">
+            <material>Gazebo/Red</material>
+        </gazebo>
         <joint name="gantry_to_support_${postfix}" type="fixed">
             <parent link="gantry"/>

Commit message: switch to action control

File: jetleg_description/urdf/jetleg.xacro (robot description, xacro)
@@ -60,5 +60,5 @@
             <child link="shank${identifier}"/>
             <axis xyz="0 1 0"/>
-            <limit effort="100" lower="0.0" upper="2.5" velocity="10"/>
+            <limit effort="10000" lower="0.0" upper="2.5" velocity="10"/>
         </joint>
         <link name="foot${identifier}">
@@ -93,5 +93,5 @@
             <child link="foot${identifier}"/>
             <axis xyz="0 1 0"/>
-            <limit effort="100" lower="-0.1" upper="0.5" velocity="10"/>
+            <limit effort="10000" lower="-0.1" upper="0.5" velocity="10"/>
         </joint>
     </xacro:macro>

File: jetleg_description/urdf/jetleg_wheeled_testrig.xacro (robot description, xacro)
@@ -88,5 +88,5 @@
         <parent link="vertical_rail"/>
         <child link="mount"/>
-        <limit effort="100" lower="${-mount_angle_lim}" upper="${mount_angle_lim}" velocity="10"/>
+        <limit effort="10000" lower="${-mount_angle_lim}" upper="${mount_angle_lim}" velocity="10"/>
         <axis xyz="0 1 0"/>
     </joint>
@@ -95,5 +95,5 @@
         <parent link="vertical_rail"/>
         <child link="mount_intact"/>
-        <limit effort="100" lower="${-mount_angle_lim}" upper="${mount_angle_lim}" velocity="10"/>
+        <limit effort="10000" lower="${-mount_angle_lim}" upper="${mount_angle_lim}" velocity="10"/>
         <axis xyz="0 1 0"/>
     </joint>

Commit message: fix control of main leg in gazebo simulation

File: jetleg_description/urdf/jetleg.xacro (robot description, xacro)
@@ -60,5 +60,5 @@
             <child link="shank${identifier}"/>
             <axis xyz="0 1 0"/>
-            <limit effort="10000" lower="0.0" upper="2.5" velocity="10"/>
+            <limit effort="100" lower="0.0" upper="2.5" velocity="10"/>
         </joint>
         <link name="foot${identifier}">
@@ -93,5 +93,5 @@
             <child link="foot${identifier}"/>
             <axis xyz="0 1 0"/>
-            <limit effort="10000" lower="-0.1" upper="0.5" velocity="10"/>
+            <limit effort="100" lower="-0.1" upper="0.5" velocity="10"/>
         </joint>
     </xacro:macro>

File: jetleg_description/urdf/jetleg_testrig.xacro (robot description, xacro)
@@ -28,5 +28,5 @@
         <origin xyz="0 0 ${-thigh_length/2}" rpy="0 0 0"/>
         <axis xyz="0 0 -1" />
-        <limit effort="1000" velocity="10" lower="0" upper="0.6" />
+        <limit effort="100" velocity="10" lower="0" upper="0.6" />
     </joint>
 </robot>

File: jetleg_description/urdf/jetleg_wheeled_testrig.xacro (robot description, xacro)
@@ -88,5 +88,5 @@
         <parent link="vertical_rail"/>
         <child link="mount"/>
-        <limit effort="10000" lower="${-mount_angle_lim}" upper="${mount_angle_lim}" velocity="10"/>
+        <limit effort="100" lower="${-mount_angle_lim}" upper="${mount_angle_lim}" velocity="10"/>
         <axis xyz="0 1 0"/>
     </joint>
@@ -95,5 +95,5 @@
         <parent link="vertical_rail"/>
         <child link="mount_intact"/>
-        <limit effort="10000" lower="${-mount_angle_lim}" upper="${mount_angle_lim}" velocity="10"/>
+        <limit effort="100" lower="${-mount_angle_lim}" upper="${mount_angle_lim}" velocity="10"/>
         <axis xyz="0 1 0"/>
     </joint>
@@ -103,5 +103,5 @@
         <origin xyz="0 0 ${-thigh_length/2}" rpy="0 0 0"/>
         <axis xyz="0 0 -1" />
-        <limit effort="1000" velocity="10" lower="0" upper="0.6" />
+        <limit effort="100" velocity="10" lower="0" upper="0.6" />
     </joint>
     <joint name="mount_to_jetleg_intact" type="fixed">
@@ -110,5 +110,5 @@
         <origin xyz="0 0 ${-thigh_length/2}" rpy="0 0 0"/>
         <axis xyz="0 0 -1" />
-        <limit effort="1000" velocity="10" lower="0" upper="0.6" />
+        <limit effort="100" velocity="10" lower="0" upper="0.6" />
     </joint>
 </robot>

File: jetleg_description/urdf/testrig.xacro (robot description, xacro)
@@ -76,5 +76,5 @@
         <parent link="gantry"/>
         <child link="vertical_rail"/>
-        <limit effort="100" lower="-1" upper="3" velocity="10"/>
+        <limit effort="100" lower="-0.5" upper="0.0" velocity="10"/>
         <axis xyz="0 0 1"/>
     </joint>

Commit message: use moveit2 to directly control trajectory

File: jetleg_description/urdf/jetleg.xacro (robot description, xacro)
@@ -97,6 +97,6 @@
         </joint>
         <!-- Import control_xacro -->
-        <xacro:include filename="$(find jetleg_description)/ros2_control/jetleg.ros2_control.xacro" />
-        <xacro:jetleg_ros2_control name="GazeboSystem" initial_positions_file="$(arg jetleg_initial_positions_file)" joint_label="${identifier}"/>
+        <!-- <xacro:include filename="$(find jetleg_description)/ros2_control/jetleg.ros2_control.xacro" />
+        <xacro:jetleg_ros2_control name="GazeboSystem" initial_positions_file="$(arg jetleg_initial_positions_file)" joint_label="${identifier}"/> -->
     </xacro:macro>
 </robot>

File: jetleg_description/urdf/jetleg_wheeled_testrig.xacro (robot description, xacro)
@@ -114,5 +114,5 @@
     <xacro:arg name="initial_positions_file" default="$(find jetleg_description)/ros2_control/initial_positions.yaml" />
     <!-- Import control_xacro -->
-    <xacro:include filename="$(find jetleg_description)/ros2_control/jetleg_wheeled_testrig.ros2_control.xacro" />
+    <!-- <xacro:include filename="$(find jetleg_description)/ros2_control/jetleg_wheeled_testrig.ros2_control.xacro" />
     <xacro:jetleg_wheeled_testrig_ros2_control name="GazeboSystem" initial_positions_file="$(arg initial_positions_file)"/>
     <gazebo>
@@ -122,4 +122,4 @@
             <robot_param_node>robot_state_publisher</robot_param_node>
         </plugin>
-    </gazebo>
+    </gazebo> -->
 </robot>

File: jetleg_description/urdf/testrig.xacro (robot description, xacro)
@@ -80,5 +80,5 @@
     </joint>
     <!-- Import control_xacro -->
-    <xacro:include filename="$(find jetleg_description)/ros2_control/testrig.ros2_control.xacro" />
-    <xacro:testrig_ros2_control name="GazeboSystem" />
+    <!-- <xacro:include filename="$(find jetleg_description)/ros2_control/testrig.ros2_control.xacro" />
+    <xacro:testrig_ros2_control name="GazeboSystem" /> -->
 </robot>

File: jetleg_moveit_config/config/jetleg_wheeled_testrig.ros2_control.xacro (robot description, xacro)
@@ -22,4 +22,11 @@
                 <state_interface name="velocity"/>
             </joint>
+            <joint name="ankle_joint">
+                <command_interface name="position"/>
+                <state_interface name="position">
+                  <param name="initial_value">${initial_positions['ankle_joint']}</param>
+                </state_interface>
+                <state_interface name="velocity"/>
+            </joint>
             <joint name="vertical_rail_to_mount_intact">
                 <command_interface name="position"/>
@@ -36,11 +43,4 @@
                 <state_interface name="velocity"/>
             </joint>
-            <joint name="ankle_joint">
-                <command_interface name="position"/>
-                <state_interface name="position">
-                  <param name="initial_value">${initial_positions['ankle_joint']}</param>
-                </state_interface>
-                <state_interface name="velocity"/>
-            </joint>
             <joint name="ankle_joint_intact">
                 <command_interface name="position"/>

Commit message: [Config] Reduce simulated leg mass

File: jetleg_description/urdf/jetleg.xacro (robot description, xacro)
@@ -8,6 +8,6 @@
     <xacro:property name="foot_width" value="0.1" />
     <xacro:property name="foot_height" value="0.05" />
-    <xacro:property name="thigh_mass" value="20" />
-    <xacro:property name="shank_mass" value="10" />
+    <xacro:property name="thigh_mass" value="1" />
+    <xacro:property name="shank_mass" value="1" />
     <xacro:property name="foot_mass" value="1.5" />
     <xacro:macro name="jetleg" params="identifier">
