Commit message: rename wheel joints to remove name conflict

File: jetleg_description/urdf/jetleg_wheeled_testrig.xacro (robot description, xacro)
@@ -33,5 +33,5 @@
             </inertial>
         </link>
-        <joint name="wheel_${wheelpos}" type="continuous">
+        <joint name="wheel_${wheelpos}_joint" type="continuous">
             <parent link="support_${parentsupport}" />
             <child link="wheel_${wheelpos}" />

Commit message: [Config] Add an imu sensor compatible with Gazebo

File: jetleg_description/urdf/jetleg_wheeled_testrig.xacro (robot description, xacro)
@@ -119,3 +119,10 @@
         </plugin>
     </gazebo>
+    <xacro:include filename="$(find jetleg_description)/urdf/jetleg_imu.xacro"/>
+    <xacro:jetleg_imu />
+    <joint name="shank_imu_joint" type="fixed">
+        <parent link="shank"/>
+        <child link="shank_imu"/>
+        <origin xyz="0 0 ${-thigh_length/2-knee_joint_radius}" rpy="0 0 0"/>
+    </joint>
 </robot>
