Commit message: Move moveit configuration to new package

File: jetleg_description/urdf/jetleg_testrig.xacro (robot description, xacro)
@@ -10,4 +10,7 @@
                 <cylinder length="${mount_length}" radius="0.08"/>
             </geometry>
+            <collision>
+                <cylinder length="${mount_length}" radius="0.08"/>
+            </collision>
             <material name="white_transluscent"/>
         </visual>

File: jetleg_description/urdf/jetleg_wheeled_testrig.xacro (robot description, xacro)
@@ -58,4 +58,9 @@
             <material name="white_transluscent"/>
         </visual>
+        <collision>
+            <geometry>
+                <cylinder length="${mount_length}" radius="0.08"/>
+            </geometry>
+        </collision>
         <inertial>
                 <mass value="1"/>
@@ -71,4 +76,9 @@
             <material name="white_transluscent"/>
         </visual>
+        <collision>
+            <geometry>
+                <cylinder length="${mount_length}" radius="0.08"/>
+            </geometry>
+        </collision>
         <inertial>
                 <mass value="1"/>

File: jetleg_description/urdf/testrig.xacro (robot description, xacro)
@@ -15,4 +15,9 @@
             <material name="white"/>
         </visual>
+        <collision>
+            <geometry>
+                <box size="0.1 0.1 0.1"/>
+            </geometry>
+        </collision>
         <inertial>
             <mass value="30"/>
@@ -27,4 +32,9 @@
             <material name="white_transluscent"/>
         </visual>
+        <collision>
+            <geometry>
+                <box size="0.05 ${gantry_width} 0.05"/>
+            </geometry>
+        </collision>
     </link>
     <xacro:macro name="support" params="postfix reflect">

File: wheeled_testrig_moveit_config/config/jetleg_wheeled_testrig.ros2_control.xacro (robot description, xacro)
@@ -5,4 +5,5 @@
         <ros2_control name="${name}" type="system">
             <hardware>
+                <!-- By default, set up controllers for simulation. This won't work on real hardware -->
                 <plugin>gazebo_ros2_control/GazeboSystem</plugin>
             </hardware>
@@ -12,5 +13,7 @@
                   <param name="initial_value">${initial_positions['vertical_rail_to_mount']}</param>
                 </state_interface>
-                <state_interface name="velocity"/>
+                <state_interface name="velocity">
+                  <param name="initial_value">0.0</param>
+                </state_interface>
             </joint>
             <joint name="knee_joint">
@@ -19,5 +22,7 @@
                   <param name="initial_value">${initial_positions['knee_joint']}</param>
                 </state_interface>
-                <state_interface name="velocity"/>
+                <state_interface name="velocity">
+                  <param name="initial_value">0.0</param>
+                </state_interface>
             </joint>
             <joint name="ankle_joint">
@@ -26,5 +31,7 @@
                   <param name="initial_value">${initial_positions['ankle_joint']}</param>
                 </state_interface>
-                <state_interface name="velocity"/>
+                <state_interface name="velocity">
+                  <param name="initial_value">0.0</param>
+                </state_interface>
             </joint>
             <joint name="vertical_rail_to_mount_intact">
@@ -33,5 +40,7 @@
                   <param name="initial_value">${initial_positions['vertical_rail_to_mount_intact']}</param>
                 </state_interface>
-                <state_interface name="velocity"/>
+                <state_interface name="velocity">
+                  <param name="initial_value">0.0</param>
+                </state_interface>
             </joint>
             <joint name="knee_joint_intact">
@@ -40,5 +49,7 @@
                   <param name="initial_value">${initial_positions['knee_joint_intact']}</param>
                 </state_interface>
-                <state_interface name="velocity"/>
+                <state_interface name="velocity">
+                  <param name="initial_value">0.0</param>
+                </state_interface>
             </joint>
             <joint name="ankle_joint_intact">
@@ -47,5 +58,7 @@
                   <param name="initial_value">${initial_positions['ankle_joint_intact']}</param>
                 </state_interface>
-                <state_interface name="velocity"/>
+                <state_interface name="velocity">
+                  <param name="initial_value">0.0</param>
+                </state_interface>
             </joint>
         </ros2_control>

Commit message: Reorganize robot description files

File: jetleg_description/urdf/jetleg_testrig.xacro (robot description, xacro)
@@ -13,7 +13,4 @@
         </visual>
     </link>
-    <gazebo reference="mount">
-        <material>Gazebo/Black</material>
-    </gazebo>
     <joint name="vertical_rail_to_mount" type="revolute">
         <origin rpy="0 0 0" xyz="0 0 0"/>

File: jetleg_description/urdf/jetleg_testrig_vision.xacro (robot description, xacro)
@@ -2,5 +2,5 @@
 <robot xmlns:xacro="http://www.ros.org/wiki/xacro" name="jetleg_testrig_vision">
   <xacro:include filename="$(find jetleg_description)/urdf/jetleg_wheeled_testrig.xacro"/>
-  <xacro:include filename="$(find jetleg_description)/urdf/stereo_camera.xacro"/>
+  <xacro:include filename="$(find jetleg_description)/urdf/components/stereo_camera.xacro"/>
   <xacro:stereo_camera baseline="0.1">
       <joint name="gantry_to_camera_base" type="fixed">

File: jetleg_description/urdf/jetleg_wheeled_testrig.xacro (robot description, xacro)
@@ -119,10 +119,3 @@
         </plugin>
     </gazebo>
-    <xacro:include filename="$(find jetleg_description)/urdf/jetleg_imu.xacro"/>
-    <xacro:jetleg_imu />
-    <joint name="shank_imu_joint" type="fixed">
-        <parent link="shank"/>
-        <child link="shank_imu"/>
-        <origin xyz="0 0 ${-thigh_length/2-knee_joint_radius}" rpy="0 0 0"/>
-    </joint>
 </robot>
