Commit message: [Config] Add inertial info to base_link in standalone jetleg model

File: jetleg_description/urdf/jetleg_standalone.xacro (robot description, xacro)
@@ -2,8 +2,13 @@
 <robot xmlns:xacro="http://www.ros.org/wiki/xacro" name="jetleg_testrig">
     <link name="base_link">
+        <!-- Gazebo requires inertial information for each link -->
+        <inertial>
+            <mass value="1"/>
+            <inertia ixx="1" ixy="0" ixz="0" iyy="1" iyz="0" izz="1"/>
+        </inertial>
     </link>
     <!-- Include the JetLeg -->
     <xacro:include filename="$(find jetleg_description)/urdf/jetleg.xacro"/>
-    <!-- Create two JetLegs -->
+    <!-- Create a JetLeg -->
     <xacro:jetleg identifier="">
     </xacro:jetleg>
