Commit message: remove superfluous robot descriptions

File: jetleg_description/ros2_control/jetleg_wheeled_testrig.ros2_control.xacro (robot description, xacro)
@@ -26,53 +26,4 @@
         </state_interface>
       </joint>
-      <!-- Passive Joints -->
-      <joint name="wheel_hind_left_joint">
-          <state_interface name="position">
-            <param name="initial_value">${initial_positions['wheel_hind_left_joint']}</param>
-          </state_interface>
-          <state_interface name="velocity">
-            <param name="initial_value">0.0</param>
-          </state_interface>
-      </joint>
-      <joint name="wheel_hind_right_joint">
-          <state_interface name="position">
-            <param name="initial_value">${initial_positions['wheel_hind_right_joint']}</param>
-          </state_interface>
-          <state_interface name="velocity">
-            <param name="initial_value">0.0</param>
-          </state_interface>
-      </joint>
-      <joint name="wheel_fore_left_joint">
-          <state_interface name="position">
-            <param name="initial_value">${initial_positions['wheel_fore_left_joint']}</param>
-          </state_interface>
-          <state_interface name="velocity">
-            <param name="initial_value">0.0</param>
-          </state_interface>
-      </joint>
-      <joint name="wheel_fore_right_joint">
-          <state_interface name="position">
-            <param name="initial_value">${initial_positions['wheel_fore_right_joint']}</param>
-          </state_interface>
-          <state_interface name="velocity">
-            <param name="initial_value">0.0</param>
-          </state_interface>
-      </joint>
-      <joint name="base_to_gantry">
-          <state_interface name="position">
-            <param name="initial_value">${initial_positions['base_to_gantry']}</param>
-          </state_interface>
-          <state_interface name="velocity">
-            <param name="initial_value">0.0</param>
-          </state_interface>
-      </joint>
-      <joint name="gantry_to_vertical_rail">
-          <state_interface name="position">
-            <param name="initial_value">${initial_positions['gantry_to_vertical_rail']}</param>
-          </state_interface>
-          <state_interface name="velocity">
-            <param name="initial_value">0.0</param>
-          </state_interface>
-      </joint>
     </ros2_control>
   </xacro:macro>

File: jetleg_description/urdf/jetleg_testrig_vision.xacro (robot description, xacro)
@@ -1,5 +1,5 @@
 <?xml version="1.0"?>
 <robot xmlns:xacro="http://www.ros.org/wiki/xacro" name="jetleg_testrig_vision">
-  <xacro:include filename="$(find jetleg_description)/urdf/jetleg_wheeled_testrig.urdf.xacro"/>
+  <xacro:include filename="$(find jetleg_description)/urdf/jetleg_wheeled_testrig.xacro"/>
   <xacro:include filename="$(find jetleg_description)/urdf/stereo_camera.xacro"/>
   <xacro:stereo_camera baseline="0.1">

File: jetleg_description/urdf/jetleg_wheeled_testrig.xacro (robot description, xacro)
@@ -112,3 +112,14 @@
         <limit effort="100" velocity="10" lower="0" upper="0.6" />
     </joint>
+    <xacro:arg name="initial_positions_file" default="$(find jetleg_description)/ros2_control/initial_positions.yaml" />
+    <!-- Import control_xacro -->
+    <xacro:include filename="$(find jetleg_description)/ros2_control/jetleg_wheeled_testrig.ros2_control.xacro" />
+    <xacro:jetleg_wheeled_testrig_ros2_control name="GazeboSystem" initial_positions_file="$(arg initial_positions_file)"/>
+    <gazebo>
+        <plugin filename="libgazebo_ros2_control.so" name="gazebo_ros2_control">
+            <parameters>$(find jetleg_description)/ros2_control/ros2_controllers.yaml</parameters>
+            <robot_param>robot_description</robot_param>
+            <robot_param_node>robot_state_publisher</robot_param_node>
+        </plugin>
+    </gazebo>
 </robot>

File: jetleg_description/urdf/testrig.xacro (robot description, xacro)
@@ -79,3 +79,6 @@
         <axis xyz="0 0 1"/>
     </joint>
+    <!-- Import control_xacro -->
+    <xacro:include filename="$(find jetleg_description)/ros2_control/testrig.ros2_control.xacro" />
+    <xacro:testrig_ros2_control name="GazeboSystem" />
 </robot>
