Commit message: [Refactor] Move Gazebo tags into separate xacro file for better clarity

File: jetleg_description/ros2_control/jetleg_testrig.urdf.xacro (robot description, xacro)
@@ -1,9 +1,11 @@
 <?xml version="1.0"?>
 <robot xmlns:xacro="http://www.ros.org/wiki/xacro" name="jetleg_testrig">
-    <xacro:arg name="initial_positions_file" default="initial_positions.yaml" />
+    <xacro:arg name="initial_positions_file" default="$(find jetleg_description)/config/initial_positions.yaml" />
     <!-- Import jetleg_testrig urdf file -->
     <xacro:include filename="$(find jetleg_description)/urdf/jetleg_testrig.xacro" />
     <!-- Import control_xacro -->
-    <xacro:include filename="jetleg_testrig.ros2_control.xacro" />
+    <xacro:include filename="$(find jetleg_description)/ros2_control/jetleg_testrig.ros2_control.xacro" />
+    <!-- Include Gazebo tags -->
+    <xacro:include filename="$(find jetleg_description)/urdf/gazebo/jetleg_testrig_gazebo.xacro" />
     <xacro:jetleg_testrig_ros2_control name="WheeledTestrigSystem" initial_positions_file="$(arg initial_positions_file)"/>
 </robot>

File: jetleg_description/urdf/jetleg_testrig.xacro (robot description, xacro)
@@ -64,7 +64,4 @@
         </inertial>
     </link>
-    <gazebo reference="mount">
-        <material>Gazebo/Black</material>
-    </gazebo>
     <link name="mount_intact">
         <visual>
@@ -80,7 +77,4 @@
         </inertial>
     </link>
-    <gazebo reference="mount_intact">
-        <material>Gazebo/Black</material>
-    </gazebo>
     <!-- Define the additional joints of the robot -->
     <joint name="vertical_rail_to_mount" type="revolute">
@@ -112,10 +106,3 @@
         <limit effort="100" velocity="10" lower="0" upper="0.6" />
     </joint>
-    <gazebo>
-        <plugin filename="libgazebo_ros2_control.so" name="gazebo_ros2_control">
-            <parameters>$(find jetleg_description)/ros2_control/ros2_controllers.yaml</parameters>
-            <robot_param>robot_description</robot_param>
-            <robot_param_node>robot_state_publisher</robot_param_node>
-        </plugin>
-    </gazebo>
 </robot>
