Commit message: [Documentation] Generate documentation for jetleg_hardware_interface

File: jetleg_description/ros2_control/jetleg_standalone.urdf.xacro (robot description, xacro)
@@ -7,4 +7,21 @@
     <!-- Import control_xacro -->
     <xacro:include filename="$(find jetleg_description)/ros2_control/jetleg.ros2_control.xacro" />
+    <!-- Import camera model -->
+    <xacro:include filename="$(find jetleg_description)/urdf/components/stereo_camera.xacro" />
     <xacro:jetleg_ros2_control name="JetlegSystem" initial_positions_file="$(arg initial_positions_file)" plugin="jetleg_system/JetlegSystem" identifier="" />
+    <gazebo>
+        <plugin filename="libgazebo_ros2_control.so" name="gazebo_ros2_control">
+            <parameters>$(find jetleg_description)/ros2_control/ros2_controllers.yaml</parameters>
+            <robot_param>robot_description</robot_param>
+            <robot_param_node>robot_state_publisher</robot_param_node>
+        </plugin>
+    </gazebo>
+    <!-- Add camera -->
+    <xacro:stereo_camera baseline="0.1">
+      <joint name="base_link_to_camera_base" type="fixed">
+          <parent link="base_link" />
+          <child link="camera_base" />
+          <origin xyz="0.1 0 0" rpy="0 ${20*pi/180} 0" />
+      </joint>
+  </xacro:stereo_camera>
 </robot>

File: jetleg_description/urdf/gazebo/jetleg_testrig_gazebo.xacro (robot description, xacro)
@@ -10,5 +10,5 @@
     <gazebo>
         <plugin filename="libgazebo_ros2_control.so" name="gazebo_ros2_control">
-            <parameters>$(find jetleg_description)/ros2_control/ros2_controllers.yaml</parameters>
+            <parameters>$(find jetleg_description)/ros2_control/ros2_controllers_standalone.yaml</parameters>
             <robot_param>robot_description</robot_param>
             <robot_param_node>robot_state_publisher</robot_param_node>

File: jetleg_description/urdf/gazebo/stereo_camera_gazebo.xacro (robot description, xacro)
@@ -49,5 +49,5 @@
                     <updateRate>0.0</updateRate>
                     <frame_name>gazebo_camera_optical_link</frame_name>
-                    <pointCloudCutoff>0.2</pointCloudCutoff>
+                    <pointCloudCutoff>0.1</pointCloudCutoff>
                     <pointCloudCutoffMax>10.0</pointCloudCutoffMax>
                     <distortionK1>0</distortionK1>
