Commit message: visualize odrive motor movement in rviz

File: jetleg_description/ros2_control/jetleg.ros2_control.xacro (robot description, xacro)
@@ -10,8 +10,20 @@
       </sensor>
       <joint name="knee_joint">
-          <param name="serial_number">000000000000</param>
-          <param name="axis">0</param>
-          <param name="enable_watchdog">1</param>
-          <param name="watchdog_timeout">0.1</param>
+        <param name="serial_number">000000000000</param>
+        <param name="axis">0</param>
+        <param name="enable_watchdog">1</param>
+        <param name="watchdog_timeout">0.1</param>
+      </joint>
+      <joint name="ankle_joint">
+        <param name="serial_number">000000000000</param>
+        <param name="axis">1</param>
+        <param name="enable_watchdog">1</param>
+        <param name="watchdog_timeout">0.1</param>
+      </joint>
+      <joint name="gantry_to_mount">
+        <param name="serial_number">000000000000</param>
+        <param name="axis">1</param>
+        <param name="enable_watchdog">1</param>
+        <param name="watchdog_timeout">0.1</param>
       </joint>
     </ros2_control>

Commit message: separate ros2_control between testrig and jetleg

File: jetleg_description/ros2_control/jetleg.ros2_control.xacro (robot description, xacro)
@@ -1,29 +1,28 @@
 <?xml version="1.0"?>
 <robot xmlns:xacro="http://www.ros.org/wiki/xacro">
-  <xacro:macro name="jetleg_ros2_control" params="name">
+  <xacro:macro name="jetleg_ros2_control" params="name initial_positions_file joint_label">
+    <xacro:property name="initial_positions" value="${load_yaml(initial_positions_file)['initial_positions']}"/>
     <ros2_control name="${name}" type="system">
       <hardware>
-        <plugin>odrive_hardware_interface/ODriveHardwareInterface</plugin>
+        <!-- By default, set up controllers for simulation. This won't work on real hardware -->
+        <plugin>gazebo_ros2_control/GazeboSystem</plugin>
       </hardware>
-      <sensor name="odrv0">
-        <param name="serial_number">000000000000</param>
-      </sensor>
-      <joint name="knee_joint">
-        <param name="serial_number">000000000000</param>
-        <param name="axis">0</param>
-        <param name="enable_watchdog">1</param>
-        <param name="watchdog_timeout">0.1</param>
+      <joint name="knee_joint${joint_label}">
+        <command_interface name="position"/>
+        <state_interface name="position">
+          <param name="initial_value">${initial_positions['knee_joint']}</param>
+        </state_interface>
+        <state_interface name="velocity">
+          <param name="initial_value">0.0</param>
+        </state_interface>
       </joint>
-      <joint name="ankle_joint">
-        <param name="serial_number">000000000000</param>
-        <param name="axis">1</param>
-        <param name="enable_watchdog">1</param>
-        <param name="watchdog_timeout">0.1</param>
-      </joint>
-      <joint name="gantry_to_mount">
-        <param name="serial_number">000000000000</param>
-        <param name="axis">1</param>
-        <param name="enable_watchdog">1</param>
-        <param name="watchdog_timeout">0.1</param>
+      <joint name="ankle_joint${joint_label}">
+        <command_interface name="position"/>
+        <state_interface name="position">
+          <param name="initial_value">${initial_positions['ankle_joint']}</param>
+        </state_interface>
+        <state_interface name="velocity">
+          <param name="initial_value">0.0</param>
+        </state_interface>
       </joint>
     </ros2_control>

File: jetleg_description/ros2_control/jetleg_wheeled_testrig.ros2_control.xacro (robot description, xacro)
@@ -1,116 +1,79 @@
 <?xml version="1.0"?>
 <robot xmlns:xacro="http://www.ros.org/wiki/xacro">
-    <xacro:macro name="jetleg_wheeled_testrig_ros2_control" params="name initial_positions_file">
-        <xacro:property name="initial_positions" value="${load_yaml(initial_positions_file)['initial_positions']}"/>
-        <ros2_control name="${name}" type="system">
-            <hardware>
-                <!-- By default, set up controllers for simulation. This won't work on real hardware -->
-                <plugin>gazebo_ros2_control/GazeboSystem</plugin>
-                <!-- <plugin>fake_components/GenericSystem</plugin> -->
-            </hardware>
-            <joint name="vertical_rail_to_mount">
-                <command_interface name="position"/>
-                <state_interface name="position">
-                  <param name="initial_value">${initial_positions['vertical_rail_to_mount']}</param>
-                </state_interface>
-                <state_interface name="velocity">
-                  <param name="initial_value">0.0</param>
-                </state_interface>
-            </joint>
-            <joint name="knee_joint">
-                <command_interface name="position"/>
-                <state_interface name="position">
-                  <param name="initial_value">${initial_positions['knee_joint']}</param>
-                </state_interface>
-                <state_interface name="velocity">
-                  <param name="initial_value">0.0</param>
-                </state_interface>
-            </joint>
-            <joint name="ankle_joint">
-                <command_interface name="position"/>
-                <state_interface name="position">
-                  <param name="initial_value">${initial_positions['ankle_joint']}</param>
-                </state_interface>
-                <state_interface name="velocity">
-                  <param name="initial_value">0.0</param>
-                </state_interface>
-            </joint>
-            <joint name="vertical_rail_to_mount_intact">
-                <command_interface name="position"/>
-                <state_interface name="position">
-                  <param name="initial_value">${initial_positions['vertical_rail_to_mount_intact']}</param>
-                </state_interface>
-                <state_interface name="velocity">
-                  <param name="initial_value">0.0</param>
-                </state_interface>
-            </joint>
-            <joint name="knee_joint_intact">
-                <command_interface name="position"/>
-                <state_interface name="position">
-                  <param name="initial_value">${initial_positions['knee_joint_intact']}</param>
-                </state_interface>
-                <state_interface name="velocity">
-                  <param name="initial_value">0.0</param>
-                </state_interface>
-            </joint>
-            <joint name="ankle_joint_intact">
-                <command_interface name="position"/>
-                <state_interface name="position">
-                  <param name="initial_value">${initial_positions['ankle_joint_intact']}</param>
-                </state_interface>
-                <state_interface name="velocity">
-                  <param name="initial_value">0.0</param>
-                </state_interface>
-            </joint>
-            <!-- Passive Joints -->
-            <joint name="wheel_hind_left_joint">
-                <state_interface name="position">
-                  <param name="initial_value">${initial_positions['wheel_hind_left_joint']}</param>
-                </state_interface>
-                <state_interface name="velocity">
-                  <param name="initial_value">0.0</param>
-                </state_interface>
-            </joint>
-            <joint name="wheel_hind_right_joint">
-                <state_interface name="position">
-                  <param name="initial_value">${initial_positions['wheel_hind_right_joint']}</param>
-                </state_interface>
-                <state_interface name="velocity">
-                  <param name="initial_value">0.0</param>
-                </state_interface>
-            </joint>
-            <joint name="wheel_fore_left_joint">
-                <state_interface name="position">
-                  <param name="initial_value">${initial_positions['wheel_fore_left_joint']}</param>
-                </state_interface>
-                <state_interface name="velocity">
-                  <param name="initial_value">0.0</param>
-                </state_interface>
-            </joint>
-            <joint name="wheel_fore_right_joint">
-                <state_interface name="position">
-                  <param name="initial_value">${initial_positions['wheel_fore_right_joint']}</param>
-                </state_interface>
-                <state_interface name="velocity">
-                  <param name="initial_value">0.0</param>
-                </state_interface>
-            </joint>
-            <joint name="base_to_gantry">
-                <state_interface name="position">
-                  <param name="initial_value">${initial_positions['base_to_gantry']}</param>
-                </state_interface>
-                <state_interface name="velocity">
-                  <param name="initial_value">0.0</param>
-                </state_interface>
-            </joint>
-            <joint name="gantry_to_vertical_rail">
-                <state_interface name="position">
-                  <param name="initial_value">${initial_positions['gantry_to_vertical_rail']}</param>
-                </state_interface>
-                <state_interface name="velocity">
-                  <param name="initial_value">0.0</param>
-                </state_interface>
-            </joint>
-        </ros2_control>
-    </xacro:macro>
+  <xacro:macro name="jetleg_wheeled_testrig_ros2_control" params="name initial_positions_file">
+    <xacro:property name="initial_positions" value="${load_yaml(initial_positions_file)['initial_positions']}"/>
+    <ros2_control name="${name}" type="system">
+      <hardware>
+        <!-- By default, set up controllers for simulation. This won't work on real hardware -->
+        <plugin>gazebo_ros2_control/GazeboSystem</plugin>
+      </hardware>
+      <joint name="vertical_rail_to_mount">
+        <command_interface name="position"/>
+        <state_interface name="position">
+          <param name="initial_value">${initial_positions['vertical_rail_to_mount']}</param>
+        </state_interface>
+        <state_interface name="velocity">
+          <param name="initial_value">0.0</param>
+        </state_interface>
+      </joint>
+      <joint name="vertical_rail_to_mount_intact">
+        <command_interface name="position"/>
+        <state_interface name="position">
+          <param name="initial_value">${initial_positions['vertical_rail_to_mount_intact']}</param>
+        </state_interface>
+        <state_interface name="velocity">
+          <param name="initial_value">0.0</param>
+        </state_interface>
+      </joint>
+      <!-- Passive Joints -->
+      <joint name="wheel_hind_left_joint">
+          <state_interface name="position">
+            <param name="initial_value">${initial_positions['wheel_hind_left_joint']}</param>
+          </state_interface>
+          <state_interface name="velocity">
+            <param name="initial_value">0.0</param>
+          </state_interface>
+      </joint>
+      <joint name="wheel_hind_right_joint">
+          <state_interface name="position">
+            <param name="initial_value">${initial_positions['wheel_hind_right_joint']}</param>
+          </state_interface>
+          <state_interface name="velocity">
+            <param name="initial_value">0.0</param>
+          </state_interface>
+      </joint>
+      <joint name="wheel_fore_left_joint">
+          <state_interface name="position">
+            <param name="initial_value">${initial_positions['wheel_fore_left_joint']}</param>
+          </state_interface>
+          <state_interface name="velocity">
+            <param name="initial_value">0.0</param>
+          </state_interface>
+      </joint>
+      <joint name="wheel_fore_right_joint">
+          <state_interface name="position">
+            <param name="initial_value">${initial_positions['wheel_fore_right_joint']}</param>
+          </state_interface>
+          <state_interface name="velocity">
+            <param name="initial_value">0.0</param>
+          </state_interface>
+      </joint>
+      <joint name="base_to_gantry">
+          <state_interface name="position">
+            <param name="initial_value">${initial_positions['base_to_gantry']}</param>
+          </state_interface>
+          <state_interface name="velocity">
+            <param name="initial_value">0.0</param>
+          </state_interface>
+      </joint>
+      <joint name="gantry_to_vertical_rail">
+          <state_interface name="position">
+            <param name="initial_value">${initial_positions['gantry_to_vertical_rail']}</param>
+          </state_interface>
+          <state_interface name="velocity">
+            <param name="initial_value">0.0</param>
+          </state_interface>
+      </joint>
+    </ros2_control>
+  </xacro:macro>
 </robot>

File: jetleg_description/urdf/jetleg.xacro (robot description, xacro)
@@ -11,4 +11,5 @@
     <xacro:property name="shank_mass" value="10" />
     <xacro:property name="foot_mass" value="1.5" />
+    <xacro:arg name="jetleg_initial_positions_file" default="$(find jetleg_description)/ros2_control/initial_positions.yaml" />
     <xacro:macro name="jetleg" params="identifier">
         <link name="thigh${identifier}">
@@ -95,4 +96,7 @@
             <limit effort="100" lower="-0.1" upper="0.5" velocity="10"/>
         </joint>
+        <!-- Import control_xacro -->
+        <xacro:include filename="$(find jetleg_description)/ros2_control/jetleg.ros2_control.xacro" />
+        <xacro:jetleg_ros2_control name="GazeboSystem" initial_positions_file="$(arg jetleg_initial_positions_file)" joint_label="${identifier}"/>
     </xacro:macro>
 </robot>

Commit message: Integrate MoveIt with Gazebo

File: jetleg_description/ros2_control/jetleg.ros2_control.xacro (robot description, xacro)
@@ -2,5 +2,5 @@
 <robot xmlns:xacro="http://www.ros.org/wiki/xacro">
   <xacro:macro name="jetleg_ros2_control" params="name initial_positions_file joint_label">
-    <xacro:property name="initial_positions" value="${load_yaml(initial_positions_file)['initial_positions']}"/>
+    <xacro:property name="initial_positions" value="${xacro.load_yaml(initial_positions_file)['initial_positions']}"/>
     <ros2_control name="${name}" type="system">
       <hardware>

File: jetleg_description/ros2_control/jetleg_wheeled_testrig.ros2_control.xacro (robot description, xacro)
@@ -2,5 +2,5 @@
 <robot xmlns:xacro="http://www.ros.org/wiki/xacro">
   <xacro:macro name="jetleg_wheeled_testrig_ros2_control" params="name initial_positions_file">
-    <xacro:property name="initial_positions" value="${load_yaml(initial_positions_file)['initial_positions']}"/>
+    <xacro:property name="initial_positions" value="${xacro.load_yaml(initial_positions_file)['initial_positions']}"/>
     <ros2_control name="${name}" type="system">
       <hardware>

File: jetleg_description/urdf/jetleg.xacro (robot description, xacro)
@@ -11,5 +11,5 @@
     <xacro:property name="shank_mass" value="10" />
     <xacro:property name="foot_mass" value="1.5" />
-    <xacro:arg name="jetleg_initial_positions_file" default="$(find jetleg_description)/ros2_control/initial_positions.yaml" />
+    <!-- <xacro:arg name="jetleg_initial_positions_file" default="$(find jetleg_description)/ros2_control/initial_positions.yaml" /> -->
     <xacro:macro name="jetleg" params="identifier">
         <link name="thigh${identifier}">
@@ -98,5 +98,5 @@
         <!-- Import control_xacro -->
         <!-- <xacro:include filename="$(find jetleg_description)/ros2_control/jetleg.ros2_control.xacro" />
-        <xacro:jetleg_ros2_control name="GazeboSystem" initial_positions_file="$(arg jetleg_initial_positions_file)" joint_label="${identifier}"/> -->
+        <xacro:jetleg_ros2_control name="Jetleg${identifier}GazeboSystem" initial_positions_file="$(arg jetleg_initial_positions_file)" joint_label="${identifier}"/> -->
     </xacro:macro>
 </robot>

File: jetleg_description/urdf/jetleg_wheeled_testrig.xacro (robot description, xacro)
@@ -112,14 +112,14 @@
         <limit effort="100" velocity="10" lower="0" upper="0.6" />
     </joint>
-    <xacro:arg name="initial_positions_file" default="$(find jetleg_description)/ros2_control/initial_positions.yaml" />
+    <!-- <xacro:arg name="initial_positions_file" default="$(find jetleg_description)/ros2_control/initial_positions.yaml" /> -->
     <!-- Import control_xacro -->
     <!-- <xacro:include filename="$(find jetleg_description)/ros2_control/jetleg_wheeled_testrig.ros2_control.xacro" />
-    <xacro:jetleg_wheeled_testrig_ros2_control name="GazeboSystem" initial_positions_file="$(arg initial_positions_file)"/>
+    <xacro:jetleg_wheeled_testrig_ros2_control name="JetlegTestrigGazeboSystem" initial_positions_file="$(arg initial_positions_file)"/> -->
     <gazebo>
         <plugin filename="libgazebo_ros2_control.so" name="gazebo_ros2_control">
-            <parameters>$(find jetleg_description)/ros2_control/ros2_controllers.yaml</parameters>
+            <parameters>$(find jetleg_moveit_config)/config/ros2_controllers.yaml</parameters>
             <robot_param>robot_description</robot_param>
             <robot_param_node>robot_state_publisher</robot_param_node>
         </plugin>
-    </gazebo> -->
+    </gazebo>
 </robot>

File: jetleg_description/urdf/testrig.xacro (robot description, xacro)
@@ -81,4 +81,4 @@
     <!-- Import control_xacro -->
     <!-- <xacro:include filename="$(find jetleg_description)/ros2_control/testrig.ros2_control.xacro" />
-    <xacro:testrig_ros2_control name="GazeboSystem" /> -->
+    <xacro:testrig_ros2_control name="TestrigGazeboSystem" /> -->
 </robot>

File: jetleg_moveit_config/config/jetleg_wheeled_testrig.ros2_control.xacro (robot description, xacro)
@@ -2,9 +2,10 @@
 <robot xmlns:xacro="http://www.ros.org/wiki/xacro">
     <xacro:macro name="jetleg_wheeled_testrig_ros2_control" params="name initial_positions_file">
-        <xacro:property name="initial_positions" value="${load_yaml(initial_positions_file)['initial_positions']}"/>
+        <xacro:property name="initial_positions" value="${xacro.load_yaml(initial_positions_file)['initial_positions']}"/>
         <ros2_control name="${name}" type="system">
             <hardware>
                 <!-- By default, set up controllers for simulation. This won't work on real hardware -->
-                <plugin>mock_components/GenericSystem</plugin>
+                <plugin>gazebo_ros2_control/GazeboSystem</plugin>
+                <!-- <plugin>mock_components/GenericSystem</plugin> -->
             </hardware>
             <joint name="vertical_rail_to_mount">
@@ -50,4 +51,45 @@
                 <state_interface name="velocity"/>
             </joint>
+            <!-- Passive Joints -->
+            <joint name="wheel_hind_left_joint">
+                <state_interface name="position">
+                  <param name="initial_value">0.0</param>
+                </state_interface>
+                <state_interface name="velocity">
+                  <param name="initial_value">0.0</param>
+                </state_interface>
+            </joint>
+            <joint name="wheel_hind_right_joint">
+                <state_interface name="position">
+                  <param name="initial_value">0.0</param>
+                </state_interface>
+                <state_interface name="velocity">
+                  <param name="initial_value">0.0</param>
+                </state_interface>
+            </joint>
+            <joint name="wheel_fore_left_joint">
+                <state_interface name="position">
+                  <param name="initial_value">0.0</param>
+                </state_interface>
+                <state_interface name="velocity">
+                  <param name="initial_value">0.0</param>
+                </state_interface>
+            </joint>
+            <joint name="wheel_fore_right_joint">
+                <state_interface name="position">
+                  <param name="initial_value">0.0</param>
+                </state_interface>
+                <state_interface name="velocity">
+                  <param name="initial_value">0.0</param>
+                </state_interface>
+            </joint>
+            <joint name="gantry_to_vertical_rail">
+                <state_interface name="position">
+                  <param name="initial_value">0.0</param>
+                </state_interface>
+                <state_interface name="velocity">
+                  <param name="initial_value">0.0</param>
+                </state_interface>
+            </joint>
         </ros2_control>
     </xacro:macro>

File: jetleg_moveit_config/config/jetleg_wheeled_testrig.urdf.xacro (robot description, xacro)
@@ -6,4 +6,4 @@
     <!-- Import control_xacro -->
     <xacro:include filename="jetleg_wheeled_testrig.ros2_control.xacro" />
-    <xacro:jetleg_wheeled_testrig_ros2_control name="FakeSystem" initial_positions_file="$(arg initial_positions_file)"/>
+    <xacro:jetleg_wheeled_testrig_ros2_control name="GazeboSystem" initial_positions_file="$(arg initial_positions_file)"/>
 </robot>
