Commit message: [Refactor] Rename wheeled testrig robot description to shorter name

File: jetleg_description/ros2_control/jetleg.ros2_control.xacro (robot description, xacro)
@@ -1,12 +1,11 @@
 <?xml version="1.0"?>
 <robot xmlns:xacro="http://www.ros.org/wiki/xacro">
-    <xacro:macro name="jetleg_ros2_control" params="name initial_positions_file">
+    <xacro:macro name="jetleg_ros2_control" params="name initial_positions_file identifier plugin">
         <xacro:property name="initial_positions" value="${xacro.load_yaml(initial_positions_file)['initial_positions']}"/>
-        <ros2_control name="${name}" type="system">
+        <ros2_control name="${name}_${identifier}" type="system">
             <hardware>
-                <plugin>gazebo_ros2_control/GazeboSystem</plugin>
-                <!-- <plugin>fake_effort_interface/GenericSystem</plugin> -->
+                <plugin>${plugin}</plugin>
             </hardware>
-            <joint name="vertical_rail_to_mount">
+            <joint name="vertical_rail_to_mount${identifier}">
                 <command_interface name="position"/>
                 <state_interface name="position">
@@ -15,5 +14,5 @@
                 <state_interface name="velocity"/>
             </joint>
-            <joint name="knee_joint">
+            <joint name="knee_joint${identifier}">
                 <command_interface name="effort"/>
                 <state_interface name="position">
@@ -22,5 +21,5 @@
                 <state_interface name="velocity"/>
             </joint>
-            <joint name="ankle_joint">
+            <joint name="ankle_joint${identifier}">
                 <command_interface name="effort"/>
                 <state_interface name="position">

File: jetleg_description/ros2_control/jetleg_testrig.ros2_control.xacro (robot description, xacro)
@@ -2,35 +2,15 @@
 <robot xmlns:xacro="http://www.ros.org/wiki/xacro">
     <xacro:arg name="initial_positions_file" default="initial_positions.yaml" />
+    <xacro:arg name="plugin" default="gazebo_ros2_control/GazeboSystem" />
     <!-- Import the JetLeg ros2_control hardware configurations -->
     <xacro:include filename="$(find jetleg_description)/ros2_control/jetleg.ros2_control.xacro" />
-    <xacro:jetleg_ros2_control name="JetlegSystem" initial_positions_file="$(arg initial_positions_file)" />
-    <xacro:macro name="jetleg_wheeled_testrig_ros2_control" params="name initial_positions_file">
+    <xacro:jetleg_ros2_control name="JetlegSystem" identifier="" initial_positions_file="$(arg initial_positions_file)" plugin="$(arg plugin)" />
+    <xacro:jetleg_ros2_control name="JetlegSystem" identifier="_intact" initial_positions_file="$(arg initial_positions_file)" plugin="$(arg plugin)" />
+    <xacro:macro name="jetleg_testrig_ros2_control" params="name initial_positions_file">
         <xacro:property name="initial_positions" value="${xacro.load_yaml(initial_positions_file)['initial_positions']}"/>
         <ros2_control name="${name}" type="system">
             <hardware>
-                <plugin>gazebo_ros2_control/GazeboSystem</plugin>
-                <!-- <plugin>fake_effort_interface/GenericSystem</plugin> -->
+                <plugin>$(arg plugin)</plugin>
             </hardware>
-            <joint name="vertical_rail_to_mount_intact">
-                <command_interface name="effort"/>
-                <state_interface name="position">
-                  <param name="initial_value">${initial_positions['vertical_rail_to_mount_intact']}</param>
-                </state_interface>
-                <state_interface name="velocity"/>
-            </joint>
-            <joint name="knee_joint_intact">
-                <command_interface name="effort"/>
-                <state_interface name="position">
-                  <param name="initial_value">${initial_positions['knee_joint_intact']}</param>
-                </state_interface>
-                <state_interface name="velocity"/>
-            </joint>
-            <joint name="ankle_joint_intact">
-                <command_interface name="effort"/>
-                <state_interface name="position">
-                  <param name="initial_value">${initial_positions['ankle_joint_intact']}</param>
-                </state_interface>
-                <state_interface name="velocity"/>
-            </joint>
             <!-- Passive Joints -->
             <joint name="wheel_hind_left_joint">
@@ -66,12 +46,4 @@
                 </state_interface>
             </joint>
-            <!-- <joint name="gantry_to_vertical_rail">
-                <state_interface name="position">
-                  <param name="initial_value">0.0</param>
-                </state_interface>
-                <state_interface name="velocity">
-                  <param name="initial_value">0.0</param>
-                </state_interface>
-            </joint> -->
         </ros2_control>
     </xacro:macro>

File: jetleg_description/urdf/jetleg.xacro (robot description, xacro)
@@ -29,7 +29,4 @@
         </inertial>
         </link>
-        <gazebo reference="thigh${identifier}">
-            <material>Gazebo/White</material>
-        </gazebo>
         <link name="shank${identifier}">
             <visual>
@@ -52,7 +49,4 @@
             </inertial>
         </link>
-        <gazebo reference="shank${identifier}">
-            <material>Gazebo/White</material>
-        </gazebo>
         <joint name="knee_joint${identifier}" type="revolute">
             <origin rpy="0 0 0" xyz="0 0 ${-thigh_length/2-knee_joint_radius}"/>
@@ -85,7 +79,4 @@
             </inertial>
         </link>
-        <gazebo reference="foot${identifier}">
-            <material>Gazebo/White</material>
-        </gazebo>
         <joint name="ankle_joint${identifier}" type="revolute">
             <origin rpy="0 0 0" xyz="0 0 ${-(knee_joint_radius + shank_length + ankle_joint_radius)}"/>

File: jetleg_description/urdf/jetleg_testrig.xacro (robot description, xacro)
@@ -1,8 +1,54 @@
 <?xml version="1.0"?>
 <robot xmlns:xacro="http://www.ros.org/wiki/xacro" name="jetleg_testrig">
+    <!-- Include the basic testrig -->
     <xacro:include filename="$(find jetleg_description)/urdf/testrig.xacro"/>
-    <xacro:include filename="jetleg.xacro"/>
+    <!-- Include the JetLeg -->
+    <xacro:include filename="$(find jetleg_description)/urdf/jetleg.xacro"/>
+    <!-- Define reusable variables -->
+    <xacro:property name="wheel_length" value="0.04" />
+    <xacro:property name="wheel_radius" value="0.15" />
+    <xacro:property name="wheel_offset" value="0.4" />
+    <!-- Define the wheel macro -->
+    <xacro:macro name="wheel" params="wheelpos parentsupport reflect offset">
+        <link name="wheel_${wheelpos}">
+            <contact>
+                <rolling_friction value="0.001"/>
+                <spinning_friction value="0.001"/>
+            </contact>
+            <visual>
+                <geometry>
+                    <cylinder length="${wheel_length}" radius="${wheel_radius}" />
+                </geometry>
+                <material name="white" />
+            </visual>
+            <collision>
+                <geometry>
+                    <cylinder length="${wheel_length}" radius="${wheel_radius}" />
+                </geometry>
+                <contact_coefficients mu="1.0" />
+            </collision>
+            <inertial>
+                <mass value="10"/>
+                <inertia ixx="0.001" ixy="0" ixz="0" iyy="0.001" iyz="0" izz="0.001"/>
+            </inertial>
+        </link>
+        <joint name="wheel_${wheelpos}_joint" type="continuous">
+            <parent link="support_${parentsupport}" />
+            <child link="wheel_${wheelpos}" />
+            <origin xyz="${offset} ${0.2 * reflect} -${gantry_height / 2}" rpy="1.57 0 0" />
+            <axis xyz="0 0 -1" />
+        </joint>
+    </xacro:macro>
+    <!-- Create four wheels for the testrig -->
+    <xacro:wheel wheelpos="fore_left" parentsupport="left" reflect="1" offset="${wheel_offset}" />
+    <xacro:wheel wheelpos="fore_right" parentsupport="right" reflect="-1" offset="${wheel_offset}" />
+    <xacro:wheel wheelpos="hind_left" parentsupport="left" reflect="1" offset="${-wheel_offset}" />
+    <xacro:wheel wheelpos="hind_right" parentsupport="right" reflect="-1" offset="${-wheel_offset}" />
+    <!-- Create two JetLegs -->
     <xacro:jetleg identifier="">
     </xacro:jetleg>
+    <xacro:jetleg identifier="_intact">
+    </xacro:jetleg>
+    <!-- Use mounts to attach legs to the testrig -->
     <link name="mount">
         <visual>
@@ -12,9 +58,41 @@
             <material name="black"/>
         </visual>
+        <inertial>
+                <mass value="1"/>
+                <inertia ixx="1" ixy="0" ixz="0" iyy="1" iyz="0" izz="1"/>
+                <origin rpy="0 0 0" xyz="0 0 0"/>
+        </inertial>
     </link>
+    <gazebo reference="mount">
+        <material>Gazebo/Black</material>
+    </gazebo>
+    <link name="mount_intact">
+        <visual>
+            <geometry>
+                <cylinder length="${mount_length}" radius="0.08"/>
+            </geometry>
+            <material name="black"/>
+        </visual>
+        <inertial>
+                <mass value="1"/>
+                <inertia ixx="1" ixy="0" ixz="0" iyy="1" iyz="0" izz="1"/>
+                <origin rpy="0 0 0" xyz="0 0 0"/>
+        </inertial>
+    </link>
+    <gazebo reference="mount_intact">
+        <material>Gazebo/Black</material>
+    </gazebo>
+    <!-- Define the additional joints of the robot -->
     <joint name="vertical_rail_to_mount" type="revolute">
-        <origin rpy="0 0 0" xyz="0 0 0"/>
+        <origin rpy="0 0 0" xyz="0 -0.1 0"/>
         <parent link="vertical_rail"/>
         <child link="mount"/>
+        <limit effort="100" lower="${-mount_angle_lim}" upper="${mount_angle_lim}" velocity="10"/>
+        <axis xyz="0 1 0"/>
+    </joint>
+    <joint name="vertical_rail_to_mount_intact" type="revolute">
+        <origin rpy="0 0 0" xyz="0 0.1 0"/>
+        <parent link="vertical_rail"/>
+        <child link="mount_intact"/>
         <limit effort="100" lower="${-mount_angle_lim}" upper="${mount_angle_lim}" velocity="10"/>
         <axis xyz="0 1 0"/>
@@ -27,3 +105,17 @@
         <limit effort="100" velocity="10" lower="0" upper="0.6" />
     </joint>
+    <joint name="mount_to_jetleg_intact" type="fixed">
+        <parent link="mount_intact"/>
+        <child link="thigh_intact"/>
+        <origin xyz="0 0 ${-thigh_length/2}" rpy="0 0 0"/>
+        <axis xyz="0 0 -1" />
+        <limit effort="100" velocity="10" lower="0" upper="0.6" />
+    </joint>
+    <gazebo>
+        <plugin filename="libgazebo_ros2_control.so" name="gazebo_ros2_control">
+            <parameters>$(find jetleg_description)/ros2_control/ros2_controllers.yaml</parameters>
+            <robot_param>robot_description</robot_param>
+            <robot_param_node>robot_state_publisher</robot_param_node>
+        </plugin>
+    </gazebo>
 </robot>

File: jetleg_description/urdf/jetleg_testrig_vision.xacro (robot description, xacro)
@@ -1,5 +1,5 @@
 <?xml version="1.0"?>
 <robot xmlns:xacro="http://www.ros.org/wiki/xacro" name="jetleg_testrig_vision">
-  <xacro:include filename="$(find jetleg_description)/urdf/jetleg_wheeled_testrig.xacro"/>
+  <xacro:include filename="$(find jetleg_description)/urdf/jetleg_testrig.xacro"/>
   <xacro:include filename="$(find jetleg_description)/urdf/components/stereo_camera.xacro"/>
   <xacro:stereo_camera baseline="0.1">

File: jetleg_description/urdf/testrig.xacro (robot description, xacro)
@@ -1,5 +1,6 @@
 <?xml version="1.0"?>
 <robot xmlns:xacro="http://www.ros.org/wiki/xacro" name="testrig">
-    <xacro:include filename="$(find jetleg_description)/urdf/colors.xacro"/>
+    <xacro:include filename="$(find jetleg_description)/urdf/colors.xacro" />
+    <xacro:include filename="$(find jetleg_description)/urdf/gazebo/testrig_gazebo.xacro" />
     <xacro:property name="gantry_height" value="1" />
     <xacro:property name="gantry_width" value="1.6" />
@@ -20,7 +21,4 @@
         </inertial>
     </link>
-    <gazebo reference="vertical_rail">
-        <material>Gazebo/White</material>
-    </gazebo>
     <link name="gantry">
         <visual>
@@ -35,7 +33,4 @@
         </inertial>
     </link>
-    <gazebo reference="gantry">
-        <material>Gazebo/White</material>
-    </gazebo>
     <xacro:macro name="support" params="postfix reflect">
         <link name="support_${postfix}">
@@ -56,7 +51,4 @@
             </inertial>
         </link>
-        <gazebo reference="support_${postfix}">
-            <material>Gazebo/Red</material>
-        </gazebo>
         <joint name="gantry_to_support_${postfix}" type="fixed">
             <parent link="gantry"/>

Commit message: [Config] Add a stand-alone leg model for testing and visualization

File: jetleg_description/ros2_control/jetleg.ros2_control.xacro (robot description, xacro)
@@ -7,11 +7,4 @@
                 <plugin>${plugin}</plugin>
             </hardware>
-            <joint name="vertical_rail_to_mount${identifier}">
-                <command_interface name="position"/>
-                <state_interface name="position">
-                  <param name="initial_value">${initial_positions['vertical_rail_to_mount']}</param>
-                </state_interface>
-                <state_interface name="velocity"/>
-            </joint>
             <joint name="knee_joint${identifier}">
                 <command_interface name="effort"/>

Commit message: [Implementation] Compute hip angle from knee angle and IMU orientation

File: jetleg_description/ros2_control/jetleg.ros2_control.xacro (robot description, xacro)
@@ -33,4 +33,12 @@
                 <state_interface name="linear_acceleration.z" />
             </sensor>
+            <!-- Use if modelling the movement of the thigh -->
+            <joint name="base_link_to_jetleg">
+                <command_interface name="effort"/>
+                <state_interface name="position">
+                    <param name="initial_value">0.0</param>
+                </state_interface>
+                <state_interface name="velocity"/>
+            </joint>
         </ros2_control>
     </xacro:macro>

File: jetleg_description/urdf/jetleg_standalone.xacro (robot description, xacro)
@@ -11,8 +11,10 @@
     <xacro:include filename="$(find jetleg_description)/urdf/components/imu.xacro" />
     <xacro:jetleg_imu />
-    <joint name="base_link_to_jetleg" type="fixed">
+    <joint name="base_link_to_jetleg" type="revolute">
         <parent link="base_link" />
         <child link="thigh" />
+        <axis xyz="0 1 0"/>
         <origin xyz="0 0 0" rpy="0 0 0" />
+        <limit effort="100" lower="0.0" upper="0.5" velocity="10"/>
     </joint>
     <!-- Define the additional joints of the robot -->
