Commit message: [Configuration] Update package versions

File: jetleg_description/ros2_control/jetleg.ros2_control.xacro (robot description, xacro)
@@ -1,23 +1,15 @@
 <?xml version="1.0"?>
 <robot xmlns:xacro="http://www.ros.org/wiki/xacro">
-    <xacro:macro name="jetleg_ros2_control" params="name initial_positions_file identifier plugin">
+    <xacro:macro name="jetleg_ros2_control" params="name initial_positions_file id plugin">
         <xacro:property name="initial_positions" value="${xacro.load_yaml(initial_positions_file)['initial_positions']}"/>
-        <ros2_control name="${name}_${identifier}" type="system">
+        <ros2_control name="${name}_${id}" type="system">
             <hardware>
                 <plugin>${plugin}</plugin>
             </hardware>
-            <joint name="knee_joint${identifier}">
+            <joint name="knee_joint_${id}">
                 <command_interface name="effort"/>
                 <state_interface name="position">
                   <param name="initial_value">${initial_positions['knee_joint']}</param>
                 </state_interface>
-                <state_interface name="velocity"/>
-            </joint>
-            <joint name="ankle_joint${identifier}">
-                <command_interface name="effort"/>
-                <state_interface name="position">
-                  <param name="initial_value">${initial_positions['ankle_joint']}</param>
-                </state_interface>
-                <state_interface name="velocity"/>
             </joint>
             <sensor name="imu0">
@@ -33,11 +25,4 @@
                 <state_interface name="linear_acceleration.z" />
             </sensor>
-            <!-- Use if modelling the movement of the thigh -->
-            <joint name="base_link_to_jetleg">
-                <state_interface name="position">
-                    <param name="initial_value">0.0</param>
-                </state_interface>
-                <state_interface name="velocity"/>
-            </joint>
         </ros2_control>
     </xacro:macro>

File: jetleg_description/ros2_control/jetleg.urdf.xacro (robot description, xacro)
@@ -1,13 +1,13 @@
 <?xml version="1.0"?>
-<robot xmlns:xacro="http://www.ros.org/wiki/xacro" name="jetleg_testrig">
+<robot xmlns:xacro="http://www.ros.org/wiki/xacro" name="jetleg">
     <xacro:arg name="initial_positions_file" default="$(find jetleg_description)/config/initial_positions.yaml" />
     <xacro:include filename="$(find jetleg_description)/urdf/colors.xacro" />
-    <!-- Import jetleg_testrig urdf file -->
-    <xacro:include filename="$(find jetleg_description)/urdf/jetleg_standalone.xacro" />
+    <!-- Import jetleg urdf file -->
+    <xacro:include filename="$(find jetleg_description)/urdf/jetleg.xacro" />
     <!-- Import control_xacro -->
     <xacro:include filename="$(find jetleg_description)/ros2_control/jetleg.ros2_control.xacro" />
     <!-- Import camera model -->
     <xacro:include filename="$(find jetleg_description)/urdf/components/stereo_camera.xacro" />
-    <xacro:jetleg_ros2_control name="JetlegSystem" initial_positions_file="$(arg initial_positions_file)" plugin="jetleg_system/JetlegSystem" identifier="" />
+    <xacro:jetleg_ros2_control name="JetlegSystem" initial_positions_file="$(arg initial_positions_file)" plugin="jetleg_system/JetlegSystem" id="" />
     <gazebo>
         <plugin filename="libgazebo_ros2_control.so" name="gazebo_ros2_control">

File: jetleg_description/urdf/components/imu.xacro (robot description, xacro)
@@ -1,4 +1,4 @@
 <?xml version="1.0"?>
-<robot xmlns:xacro="http://www.ros.org/wiki/xacro" name="imu">
+<robot xmlns:xacro="http://www.ros.org/wiki/xacro" name="imu0">
     <xacro:macro name="jetleg_imu" >
         <link name="shank_imu">
@@ -15,5 +15,5 @@
         <joint name="imu_to_shank" type="fixed">
             <origin rpy="0 0 0" xyz="0 0 -0.2" />
-            <parent link="shank" />
+            <parent link="shank_" />
             <child link="shank_imu" />
         </joint>

File: jetleg_description/urdf/jetleg.xacro (robot description, xacro)
@@ -1,89 +1,22 @@
 <?xml version="1.0"?>
 <robot xmlns:xacro="http://www.ros.org/wiki/xacro" name="jetleg">
-    <xacro:property name="thigh_length" value="0.5" />
-    <xacro:property name="shank_length" value="0.4" />
-    <xacro:property name="knee_joint_radius" value="0.025" />
-    <xacro:property name="ankle_joint_radius" value="0.025" />
-    <xacro:property name="foot_length" value="0.3" />
-    <xacro:property name="foot_width" value="0.1" />
-    <xacro:property name="foot_height" value="0.05" />
-    <xacro:property name="thigh_mass" value="1" />
-    <xacro:property name="shank_mass" value="1" />
-    <xacro:property name="foot_mass" value="1.5" />
-    <xacro:macro name="jetleg" params="identifier">
-        <link name="thigh${identifier}">
-            <visual>
-                <geometry>
-                    <cylinder length="${thigh_length}" radius="0.06"/>
-                </geometry>
-                <material name="white"/>
-            </visual>
-            <collision>
-                <geometry>
-                    <cylinder length="${thigh_length}" radius="0.06"/>
-                </geometry>
-            </collision>
-            <inertial>
-            <mass value="${thigh_mass}"/>
+    <link name="base_link">
+        <!-- Gazebo requires inertial information for each link -->
+        <inertial>
+            <mass value="1"/>
             <inertia ixx="1" ixy="0" ixz="0" iyy="1" iyz="0" izz="1"/>
         </inertial>
-        </link>
-        <link name="shank${identifier}">
-            <visual>
-                <geometry>
-                    <cylinder length="${shank_length}" radius="0.06"/>
-                </geometry>
-                <material name="white"/>
-                <origin rpy="0 0 0" xyz="0 0 ${-shank_length/2-knee_joint_radius}"/>
-            </visual>
-            <collision>
-                <geometry>
-                    <cylinder length="${shank_length}" radius="0.06"/>
-                </geometry>
-                <origin rpy="0 0 0" xyz="0 0 ${-shank_length/2-knee_joint_radius}"/>
-            </collision>
-            <inertial>
-                <mass value="${shank_mass}"/>
-                <inertia ixx="1" ixy="0" ixz="0" iyy="1" iyz="0" izz="1"/>
-                <origin rpy="0 0 0" xyz="0 0 ${-shank_length/2-knee_joint_radius}"/>
-            </inertial>
-        </link>
-        <joint name="knee_joint${identifier}" type="revolute">
-            <origin rpy="0 0 0" xyz="0 0 ${-thigh_length/2-knee_joint_radius}"/>
-            <parent link="thigh${identifier}"/>
-            <child link="shank${identifier}"/>
-            <axis xyz="0 1 0"/>
-            <limit effort="100" lower="0.0" upper="2.5" velocity="10"/>
-        </joint>
-        <link name="foot${identifier}">
-            <contact>
-                <lateral_friction value="100"/>
-            </contact>
-            <visual>
-                <geometry>
-                    <box size="${foot_length} ${foot_width} ${foot_height}"/>
-                </geometry>
-                <material name="white"/>
-                <origin xyz="${(foot_length/2-0.05)} 0 ${-ankle_joint_radius-foot_height/2}"/>
-            </visual>
-            <collision>
-                <geometry>
-                    <box size="${foot_length} ${foot_width} ${foot_height}"/>
-                </geometry>
-                <origin xyz="${(foot_length/2-0.05)} 0 ${-ankle_joint_radius-foot_height/2}"/>
-            </collision>
-            <inertial>
-                <mass value="${foot_mass}"/>
-                <inertia ixx="1" ixy="0" ixz="0" iyy="1" iyz="0" izz="1"/>
-                <origin xyz="${(foot_length/2-0.05)} 0 ${-ankle_joint_radius-foot_height/2}"/>
-            </inertial>
-        </link>
-        <joint name="ankle_joint${identifier}" type="revolute">
-            <origin rpy="0 0 0" xyz="0 0 ${-(knee_joint_radius + shank_length + ankle_joint_radius)}"/>
-            <parent link="shank${identifier}"/>
-            <child link="foot${identifier}"/>
-            <axis xyz="0 1 0"/>
-            <limit effort="100" lower="-0.1" upper="0.5" velocity="10"/>
-        </joint>
-    </xacro:macro>
+    </link>
+    <!-- Include the JetLeg -->
+    <xacro:include filename="$(find jetleg_description)/urdf/components/jetleg.macro.xacro"/>
+    <!-- Create a JetLeg -->
+    <xacro:jetleg id="">
+    </xacro:jetleg>
+    <!-- Include components -->
+    <xacro:include filename="$(find jetleg_description)/urdf/components/imu.xacro" />
+    <xacro:jetleg_imu />
+    <joint name="base_link_to_jetleg" type="fixed">
+        <parent link="base_link" />
+        <child link="thigh_" />
+    </joint>
 </robot>
