Commit message: Setup moveit_config package

File: jetleg_description/ros2_control/jetleg.urdf.xacro (robot description, xacro)
@@ -9,5 +9,5 @@
     <!-- Import camera model -->
     <xacro:include filename="$(find jetleg_description)/urdf/components/stereo_camera.xacro" />
-    <xacro:jetleg_ros2_control name="JetlegSystem" initial_positions_file="$(arg initial_positions_file)" plugin="jetleg_system/JetlegSystem" id="" />
+    <xacro:jetleg_ros2_control name="JetlegSystem" initial_positions_file="$(arg initial_positions_file)" plugin="gazebo_ros2_control/GazeboSystem" id="" />
     <gazebo>
         <plugin filename="libgazebo_ros2_control.so" name="gazebo_ros2_control">

File: jetleg_description/urdf/jetleg.xacro (robot description, xacro)
@@ -2,9 +2,4 @@
 <robot xmlns:xacro="http://www.ros.org/wiki/xacro" name="jetleg">
     <link name="base_link">
-        <!-- Gazebo requires inertial information for each link -->
-        <inertial>
-            <mass value="1"/>
-            <inertia ixx="1" ixy="0" ixz="0" iyy="1" iyz="0" izz="1"/>
-        </inertial>
     </link>
     <!-- Include the JetLeg -->
