Commit message: Add FakeSystem to test ros2_control and MoveIt functionality

File: jetleg_moveit_config/config/jetleg_wheeled_testrig.ros2_control.xacro (robot description, xacro)
@@ -2,10 +2,10 @@
 <robot xmlns:xacro="http://www.ros.org/wiki/xacro">
     <xacro:macro name="jetleg_wheeled_testrig_ros2_control" params="name initial_positions_file">
-        <xacro:property name="initial_positions" value="${xacro.load_yaml(initial_positions_file)['initial_positions']}"/>
+        <xacro:property name="initial_positions" value="${load_yaml(initial_positions_file)['initial_positions']}"/>
         <ros2_control name="${name}" type="system">
             <hardware>
                 <!-- By default, set up controllers for simulation. This won't work on real hardware -->
                 <plugin>gazebo_ros2_control/GazeboSystem</plugin>
-                <!-- <plugin>mock_components/GenericSystem</plugin> -->
+                <!-- <plugin>fake_components/GenericSystem</plugin> -->
             </hardware>
             <joint name="vertical_rail_to_mount">

Commit message: [Configuration] Switch to impedance control for testing

File: jetleg_moveit_config/config/jetleg_wheeled_testrig.ros2_control.xacro (robot description, xacro)
@@ -2,13 +2,13 @@
 <robot xmlns:xacro="http://www.ros.org/wiki/xacro">
     <xacro:macro name="jetleg_wheeled_testrig_ros2_control" params="name initial_positions_file">
-        <xacro:property name="initial_positions" value="${load_yaml(initial_positions_file)['initial_positions']}"/>
+        <xacro:property name="initial_positions" value="${xacro.load_yaml(initial_positions_file)['initial_positions']}"/>
         <ros2_control name="${name}" type="system">
             <hardware>
                 <!-- By default, set up controllers for simulation. This won't work on real hardware -->
-                <plugin>gazebo_ros2_control/GazeboSystem</plugin>
-                <!-- <plugin>fake_components/GenericSystem</plugin> -->
+                <!-- <plugin>gazebo_ros2_control/GazeboSystem</plugin> -->
+                <plugin>fake_effort_interface/GenericSystem</plugin>
             </hardware>
             <joint name="vertical_rail_to_mount">
-                <command_interface name="position"/>
+                <command_interface name="acceleration"/>
                 <state_interface name="position">
                   <param name="initial_value">${initial_positions['vertical_rail_to_mount']}</param>
@@ -17,5 +17,5 @@
             </joint>
             <joint name="knee_joint">
-                <command_interface name="position"/>
+                <command_interface name="acceleration"/>
                 <state_interface name="position">
                   <param name="initial_value">${initial_positions['knee_joint']}</param>
@@ -24,5 +24,5 @@
             </joint>
             <joint name="ankle_joint">
-                <command_interface name="position"/>
+                <command_interface name="acceleration"/>
                 <state_interface name="position">
                   <param name="initial_value">${initial_positions['ankle_joint']}</param>
@@ -31,5 +31,5 @@
             </joint>
             <joint name="vertical_rail_to_mount_intact">
-                <command_interface name="position"/>
+                <command_interface name="acceleration"/>
                 <state_interface name="position">
                   <param name="initial_value">${initial_positions['vertical_rail_to_mount_intact']}</param>
@@ -38,5 +38,5 @@
             </joint>
             <joint name="knee_joint_intact">
-                <command_interface name="position"/>
+                <command_interface name="acceleration"/>
                 <state_interface name="position">
                   <param name="initial_value">${initial_positions['knee_joint_intact']}</param>
@@ -45,5 +45,5 @@
             </joint>
             <joint name="ankle_joint_intact">
-                <command_interface name="position"/>
+                <command_interface name="acceleration"/>
                 <state_interface name="position">
                   <param name="initial_value">${initial_positions['ankle_joint_intact']}</param>
