Commit message: [Implementation] Add an imu sensor to jetleg xacro description

File: jetleg_description/urdf/components/imu.xacro (robot description, xacro)
@@ -1,4 +1,4 @@
 <?xml version="1.0"?>
-<robot xmlns:xacro="http://www.ros.org/wiki/xacro" name="testrig">
+<robot xmlns:xacro="http://www.ros.org/wiki/xacro" name="imu">
     <xacro:macro name="jetleg_imu" >
         <link name="shank_imu">
@@ -9,8 +9,13 @@
             </visual>
             <inertial>
-                <mass value="1"/>
-                <inertia ixx="1" ixy="0" ixz="0" iyy="1" iyz="0" izz="1"/>
+                <mass value="0.1"/>
+                <inertia ixx="0.1" ixy="0" ixz="0" iyy="0.1" iyz="0" izz="0.1"/>
             </inertial>
         </link>
+        <joint name="imu_to_shank" type="fixed">
+            <origin rpy="0 0 0" xyz="0 0 -0.2" />
+            <parent link="shank" />
+            <child link="shank_imu" />
+        </joint>
         <gazebo reference="shank_imu">
             <gravity>true</gravity>

File: jetleg_description/urdf/components/stereo_camera.xacro (robot description, xacro)
@@ -16,7 +16,4 @@
             </inertial>
         </link>
-        <gazebo reference="camera_base">
-            <material>Gazebo/Grey</material>
-        </gazebo>
         <!-- Links representing the lenses -->
         <link name="camera_link">
@@ -46,10 +43,4 @@
             </inertial>
         </link>
-        <gazebo reference="camera_link">
-            <material>Gazebo/Black</material>
-        </gazebo>
-        <gazebo reference="camera_link_right">
-            <material>Gazebo/Black</material>
-        </gazebo>
         <xacro:insert_block name="joint" />
         <joint name="camera_base_to_camera_link" type="fixed">
@@ -63,58 +54,6 @@
             <origin xyz="0 ${baseline/2} 0" rpy="${90*pi/180} 0 ${90*pi/180}" />
         </joint>
-        <!-- Used to align camera between Gazebo / ROS coordinate systems -->
-        <link name="gazebo_camera_link">
-        </link>
-        <joint name="gazebo_camera_joint" type="fixed">
-            <parent link="camera_link" />
-            <child link="gazebo_camera_link" />
-            <origin xyz="0 0 0" rpy="${pi/2} ${-pi/2} ${pi}" />
-        </joint>
-        <link name="gazebo_camera_optical_link">
-        </link>
-        <joint name="gazebo_camera_optical_joint" type="fixed">
-            <parent link="gazebo_camera_link" />
-            <child link="gazebo_camera_optical_link" />
-            <origin xyz="0 0 0" rpy="${-pi/2} 0 ${-pi/2}" />
-        </joint>
-        <!-- Specifies configurations for simulating in Gazebo -->
-        <gazebo reference="gazebo_camera_link">
-            <sensor name="camera" type="depth">
-                <visualize>true</visualize>
-                <update_rate>60.0</update_rate>
-                <camera name="head">
-                    <horizontal_fov>${110*pi/180}</horizontal_fov>
-                    <image>
-                        <width>1280</width>
-                        <height>720</height>
-                        <format>R8G8B8</format>
-                    </image>
-                    <clip>
-                        <near>1.0</near>
-                        <far>20</far>
-                    </clip>
-                </camera>
-                <plugin name="depth_camera_controller" filename="libgazebo_ros_camera.so">
-                    <baseline>0.2</baseline>
-                    <alwaysOn>true</alwaysOn>
-                    <updateRate>0.0</updateRate>
-                    <frame_name>gazebo_camera_optical_link</frame_name>
-                    <pointCloudCutoff>0.2</pointCloudCutoff>
-                    <pointCloudCutoffMax>10.0</pointCloudCutoffMax>
-                    <distortionK1>0</distortionK1>
-                    <distortionK2>0</distortionK2>
-                    <distortionK3>0</distortionK3>
-                    <distortionT1>0</distortionT1>
-                    <distortionT2>0</distortionT2>
-                    <CxPrime>0</CxPrime>
-                    <Cx>0</Cx>
-                    <Cy>0</Cy>
-                    <min_depth>0.1</min_depth>
-                    <max_depth>100.0</max_depth>
-                    <focalLength>0</focalLength>
-                    <hackBaseline>0</hackBaseline>
-                </plugin>
-            </sensor>
-        </gazebo>
+        <xacro:include filename="$(find jetleg_description)/urdf/gazebo/stereo_camera_gazebo.xacro" />
+        <xacro:stereo_camera_gazebo baseline="${baseline}" />
     </xacro:macro>
 </robot>

File: jetleg_description/urdf/jetleg_testrig.xacro (robot description, xacro)
@@ -77,4 +77,7 @@
         </inertial>
     </link>
+    <!-- Include components -->
+    <xacro:include filename="$(find jetleg_description)/urdf/components/imu.xacro" />
+    <xacro:jetleg_imu />
     <!-- Define the additional joints of the robot -->
     <joint name="vertical_rail_to_mount" type="revolute">
